File: SMD Emma Badge/file60C9CD01.sch (KiCad schematic (older format))
At the start: 7 parts

Commit message: Working through basics of the LFSR
Parts:
- gave numbers to parts that had none: 7
Changed lines of the file:
@@
 $Descr A4 11693 8268
 encoding utf-8
-Sheet 2 3
+Sheet 2 4
 Title ""
 Date ""
@@
 AR Path="/60B031D5/60CA0159" Ref="U?"  Part="1"
 AR Path="/60B094D9/60CA0159" Ref="U?"  Part="1"
-AR Path="/60C9CD02/60CA0159" Ref="U?"  Part="1"
-F 0 "U?" H 3650 3581 50  0000 C CNN
+AR Path="/60C9CD02/60CA0159" Ref="U201"  Part="1"
+F 0 "U201" H 3650 3581 50  0000 C CNN
 F 1 "LM555xM" H 3650 3490 50  0000 C CNN
 F 2 "Package_SO:SOIC-8_3.9x4.9mm_P1.27mm" H 4500 2600 50  0001 C CNN
@@
 AR Path="/60B031D5/60CA015F" Ref="#PWR?"  Part="1"
 AR Path="/60B094D9/60CA015F" Ref="#PWR?"  Part="1"
-AR Path="/60C9CD02/60CA015F" Ref="#PWR?"  Part="1"
-F 0 "#PWR?" H 3650 1550 50  0001 C CNN
+AR Path="/60C9CD02/60CA015F" Ref="#PWR0201"  Part="1"
+F 0 "#PWR0201" H 3650 1550 50  0001 C CNN
 F 1 "+5V" H 3665 1873 50  0000 C CNN
 F 2 "" H 3650 1700 50  0001 C CNN
@@
 AR Path="/60B031D5/60CA0166" Ref="#PWR?"  Part="1"
 AR Path="/60B094D9/60CA0166" Ref="#PWR?"  Part="1"
-AR Path="/60C9CD02/60CA0166" Ref="#PWR?"  Part="1"
-F 0 "#PWR?" H 3650 4300 50  0001 C CNN
+AR Path="/60C9CD02/60CA0166" Ref="#PWR0202"  Part="1"
+F 0 "#PWR0202" H 3650 4300 50  0001 C CNN
 F 1 "GND" H 3655 4377 50  0000 C CNN
 F 2 "" H 3650 4550 50  0001 C CNN
@@
 AR Path="/60B031D5/60CA016F" Ref="R?"  Part="1"
 AR Path="/60B094D9/60CA016F" Ref="R?"  Part="1"
-AR Path="/60C9CD02/60CA016F" Ref="R?"  Part="1"
-F 0 "R?" H 4520 2496 50  0000 L CNN
+AR Path="/60C9CD02/60CA016F" Ref="R203"  Part="1"
+F 0 "R203" H 4520 2496 50  0000 L CNN
 F 1 "1k" H 4520 2405 50  0000 L CNN
 F 2 "Resistor_SMD:R_0603_1608Metric" V 4380 2450 50  0001 C CNN
@@
 AR Path="/60B031D5/60CA017D" Ref="C?"  Part="1"
 AR Path="/60B094D9/60CA017D" Ref="C?"  Part="1"
-AR Path="/60C9CD02/60CA017D" Ref="C?"  Part="1"
-F 0 "C?" V 3898 1800 50  0000 C CNN
+AR Path="/60C9CD02/60CA017D" Ref="C203"  Part="1"
+F 0 "C203" V 3898 1800 50  0000 C CNN
 F 1 "0.1uF" V 3989 1800 50  0000 C CNN
 F 2 "Capacitor_SMD:C_0603_1608Metric" H 4188 1650 50  0001 C CNN
@@
 AR Path="/60B031D5/60CA0183" Ref="#PWR?"  Part="1"
 AR Path="/60B094D9/60CA0183" Ref="#PWR?"  Part="1"
-AR Path="/60C9CD02/60CA0183" Ref="#PWR?"  Part="1"
-F 0 "#PWR?" H 4650 1550 50  0001 C CNN
+AR Path="/60C9CD02/60CA0183" Ref="#PWR0203"  Part="1"
+F 0 "#PWR0203" H 4650 1550 50  0001 C CNN
 F 1 "GND" V 4655 1672 50  0000 R CNN
 F 2 "" H 4650 1800 50  0001 C CNN
@@
 AR Path="/60B031D5/60CA018E" Ref="C?"  Part="1"
 AR Path="/60B094D9/60CA018E" Ref="C?"  Part="1"
-AR Path="/60C9CD02/60CA018E" Ref="C?"  Part="1"
-F 0 "C?" H 2665 3946 50  0000 L CNN
+AR Path="/60C9CD02/60CA018E" Ref="C201"  Part="1"
+F 0 "C201" H 2665 3946 50  0000 L CNN
 F 1 "10u" H 2665 3855 50  0000 L CNN
 F 2 "Capacitor_SMD:C_0603_1608Metric" H 2588 3750 50  0001 C CNN
@@
 AR Path="/60B094D9/60CA01A0" Ref="R?"  Part="1"
 AR Path="/60CA01A0" Ref="R?"  Part="1"
-AR Path="/60C9CD02/60CA01A0" Ref="R?"  Part="1"
-F 0 "R?" H 2120 3196 50  0000 L CNN
+AR Path="/60C9CD02/60CA01A0" Ref="R202"  Part="1"
+F 0 "R202" H 2120 3196 50  0000 L CNN
 F 1 "11k" H 2120 3105 50  0000 L CNN
 F 2 "Resistor_SMD:R_0603_1608Metric" V 1980 3150 50  0001 C CNN
@@
 AR Path="/60B094D9/60CA01A7" Ref="R?"  Part="1"
 AR Path="/60CA01A7" Ref="R?"  Part="1"
-AR Path="/60C9CD02/60CA01A7" Ref="R?"  Part="1"
-F 0 "R?" H 2120 2596 50  0000 L CNN
+AR Path="/60C9CD02/60CA01A7" Ref="R201"  Part="1"
+F 0 "R201" H 2120 2596 50  0000 L CNN
 F 1 "11k" H 2120 2505 50  0000 L CNN
 F 2 "Resistor_SMD:R_0603_1608Metric" V 1980 2550 50  0001 C CNN
@@
 AR Path="/60B031D5/60CA01BE" Ref="C?"  Part="1"
 AR Path="/60B094D9/60CA01BE" Ref="C?"  Part="1"
-AR Path="/60C9CD02/60CA01BE" Ref="C?"  Part="1"
-F 0 "C?" H 3165 3946 50  0000 L CNN
+AR Path="/60C9CD02/60CA01BE" Ref="C202"  Part="1"
+F 0 "C202" H 3165 3946 50  0000 L CNN
 F 1 "8.2n" H 3165 3855 50  0000 L CNN
 F 2 "Capacitor_SMD:C_0603_1608Metric" H 3088 3750 50  0001 C CNN

Commit message: Routing the registers
Connections:
- net +5V: now also C203.2; no longer C203.1
- net GND: now also C203.1; no longer C203.2
Changed lines of the file:
@@
 F 4 " C14663" V 4150 1800 50  0001 C CNN "LCSC"
 	1    4150 1800
-	0    -1   -1   0
+	0    1    1    0
 $EndComp
 $Comp

Commit message: Working on letters
Parts:
- renumbered C203 to C201, C201 to C202, C202 to C203, R203 to R201, R201 to R202, R202 to R203
Changed lines of the file:
@@
 $Descr A4 11693 8268
 encoding utf-8
-Sheet 2 4
+Sheet 2 8
 Title ""
 Date ""
@@
 AR Path="/60B031D5/60CA0166" Ref="#PWR?"  Part="1"
 AR Path="/60B094D9/60CA0166" Ref="#PWR?"  Part="1"
-AR Path="/60C9CD02/60CA0166" Ref="#PWR0202"  Part="1"
-F 0 "#PWR0202" H 3650 4300 50  0001 C CNN
+AR Path="/60C9CD02/60CA0166" Ref="#PWR0203"  Part="1"
+F 0 "#PWR0203" H 3650 4300 50  0001 C CNN
 F 1 "GND" H 3655 4377 50  0000 C CNN
 F 2 "" H 3650 4550 50  0001 C CNN
@@
 AR Path="/60B031D5/60CA016F" Ref="R?"  Part="1"
 AR Path="/60B094D9/60CA016F" Ref="R?"  Part="1"
-AR Path="/60C9CD02/60CA016F" Ref="R203"  Part="1"
-F 0 "R203" H 4520 2496 50  0000 L CNN
+AR Path="/60C9CD02/60CA016F" Ref="R201"  Part="1"
+F 0 "R201" H 4520 2496 50  0000 L CNN
 F 1 "1k" H 4520 2405 50  0000 L CNN
 F 2 "Resistor_SMD:R_0603_1608Metric" V 4380 2450 50  0001 C CNN
@@
 AR Path="/60B031D5/60CA017D" Ref="C?"  Part="1"
 AR Path="/60B094D9/60CA017D" Ref="C?"  Part="1"
-AR Path="/60C9CD02/60CA017D" Ref="C203"  Part="1"
-F 0 "C203" V 3898 1800 50  0000 C CNN
+AR Path="/60C9CD02/60CA017D" Ref="C201"  Part="1"
+F 0 "C201" V 3898 1800 50  0000 C CNN
 F 1 "0.1uF" V 3989 1800 50  0000 C CNN
 F 2 "Capacitor_SMD:C_0603_1608Metric" H 4188 1650 50  0001 C CNN
@@
 AR Path="/60B031D5/60CA0183" Ref="#PWR?"  Part="1"
 AR Path="/60B094D9/60CA0183" Ref="#PWR?"  Part="1"
-AR Path="/60C9CD02/60CA0183" Ref="#PWR0203"  Part="1"
-F 0 "#PWR0203" H 4650 1550 50  0001 C CNN
+AR Path="/60C9CD02/60CA0183" Ref="#PWR0202"  Part="1"
+F 0 "#PWR0202" H 4650 1550 50  0001 C CNN
 F 1 "GND" V 4655 1672 50  0000 R CNN
 F 2 "" H 4650 1800 50  0001 C CNN
@@
 AR Path="/60B031D5/60CA018E" Ref="C?"  Part="1"
 AR Path="/60B094D9/60CA018E" Ref="C?"  Part="1"
-AR Path="/60C9CD02/60CA018E" Ref="C201"  Part="1"
-F 0 "C201" H 2665 3946 50  0000 L CNN
+AR Path="/60C9CD02/60CA018E" Ref="C202"  Part="1"
+F 0 "C202" H 2665 3946 50  0000 L CNN
 F 1 "10u" H 2665 3855 50  0000 L CNN
 F 2 "Capacitor_SMD:C_0603_1608Metric" H 2588 3750 50  0001 C CNN
@@
 AR Path="/60B094D9/60CA01A0" Ref="R?"  Part="1"
 AR Path="/60CA01A0" Ref="R?"  Part="1"
-AR Path="/60C9CD02/60CA01A0" Ref="R202"  Part="1"
-F 0 "R202" H 2120 3196 50  0000 L CNN
+AR Path="/60C9CD02/60CA01A0" Ref="R203"  Part="1"
+F 0 "R203" H 2120 3196 50  0000 L CNN
 F 1 "11k" H 2120 3105 50  0000 L CNN
 F 2 "Resistor_SMD:R_0603_1608Metric" V 1980 3150 50  0001 C CNN
@@
 AR Path="/60B094D9/60CA01A7" Ref="R?"  Part="1"
 AR Path="/60CA01A7" Ref="R?"  Part="1"
-AR Path="/60C9CD02/60CA01A7" Ref="R201"  Part="1"
-F 0 "R201" H 2120 2596 50  0000 L CNN
+AR Path="/60C9CD02/60CA01A7" Ref="R202"  Part="1"
+F 0 "R202" H 2120 2596 50  0000 L CNN
 F 1 "11k" H 2120 2505 50  0000 L CNN
 F 2 "Resistor_SMD:R_0603_1608Metric" V 1980 2550 50  0001 C CNN
@@
 AR Path="/60B031D5/60CA01BE" Ref="C?"  Part="1"
 AR Path="/60B094D9/60CA01BE" Ref="C?"  Part="1"
-AR Path="/60C9CD02/60CA01BE" Ref="C202"  Part="1"
-F 0 "C202" H 3165 3946 50  0000 L CNN
+AR Path="/60C9CD02/60CA01BE" Ref="C203"  Part="1"
+F 0 "C203" H 3165 3946 50  0000 L CNN
 F 1 "8.2n" H 3165 3855 50  0000 L CNN
 F 2 "Capacitor_SMD:C_0603_1608Metric" H 3088 3750 50  0001 C CNN
