File: SMD Emma Badge/file60CB0F51.sch (KiCad schematic (older format))
At the start: 13 parts, among them U401 74164, U402 74LS595, U403 74164, U404 74HC86, U405 74HC04

Commit message: Working on letters
Parts:
- renumbered C403 to C401, C406 to C402, C401 to C403, C402 to C406, R402 to R401, R401 to R402, U405 to U404, U404 to U405
Changed lines of the file:
@@
 $Descr A4 11693 8268
 encoding utf-8
-Sheet 4 4
+Sheet 4 8
 Title ""
 Date ""
@@
 $EndComp
 $Comp
-L power:+5V #PWR0103
+L power:+5V #PWR0402
 U 1 1 60CBA05E
 P 4900 2000
-F 0 "#PWR0103" H 4900 1850 50  0001 C CNN
+F 0 "#PWR0402" H 4900 1850 50  0001 C CNN
 F 1 "+5V" H 4915 2173 50  0000 C CNN
 F 2 "" H 4900 2000 50  0001 C CNN
@@
 Connection ~ 2900 2100
 $Comp
-L 74xx:74HC86 U404
+L 74xx:74HC86 U405
 U 1 1 60CCCFC9
 P 4300 5500
-F 0 "U404" H 4300 5825 50  0000 C CNN
+F 0 "U405" H 4300 5825 50  0000 C CNN
 F 1 "74HC86" H 4300 5734 50  0000 C CNN
 F 2 "" H 4300 5500 50  0001 C CNN
@@
 $EndComp
 $Comp
-L 74xx:74HC86 U404
+L 74xx:74HC86 U405
 U 2 1 60CCEC7D
 P 1350 7250
-F 0 "U404" H 1350 7575 50  0000 C CNN
+F 0 "U405" H 1350 7575 50  0000 C CNN
 F 1 "74HC86" H 1350 7484 50  0000 C CNN
 F 2 "" H 1350 7250 50  0001 C CNN
@@
 $EndComp
 $Comp
-L 74xx:74HC86 U404
+L 74xx:74HC86 U405
 U 3 1 60CD1561
 P 2500 6000
-F 0 "U404" H 2500 6325 50  0000 C CNN
+F 0 "U405" H 2500 6325 50  0000 C CNN
 F 1 "74HC86" H 2500 6234 50  0000 C CNN
 F 2 "" H 2500 6000 50  0001 C CNN
@@
 $EndComp
 $Comp
-L 74xx:74HC86 U404
+L 74xx:74HC86 U405
 U 4 1 60CD320B
 P 2500 5000
-F 0 "U404" H 2500 5325 50  0000 C CNN
+F 0 "U405" H 2500 5325 50  0000 C CNN
 F 1 "74HC86" H 2500 5234 50  0000 C CNN
 F 2 "" H 2500 5000 50  0001 C CNN
@@
 $EndComp
 $Comp
-L 74xx:74HC86 U404
+L 74xx:74HC86 U405
 U 5 1 60CD5100
 P 2350 7150
-F 0 "U404" H 2580 7196 50  0000 L CNN
+F 0 "U405" H 2580 7196 50  0000 L CNN
 F 1 "74HC86" H 2580 7105 50  0000 L CNN
 F 2 "Package_SO:SOIC-14_3.9x8.7mm_P1.27mm" H 2350 7150 50  0001 C CNN
@@
 $EndComp
 $Comp
-L 74xx:74HC04 U405
+L 74xx:74HC04 U404
 U 1 1 60CD8C4F
 P 8300 5300
-F 0 "U405" H 8300 5617 50  0000 C CNN
+F 0 "U404" H 8300 5617 50  0000 C CNN
 F 1 "74HC04" H 8300 5526 50  0000 C CNN
 F 2 "" H 8300 5300 50  0001 C CNN
@@
 $EndComp
 $Comp
-L 74xx:74HC04 U405
+L 74xx:74HC04 U404
 U 2 1 60CD9E44
 P 3200 5000
-F 0 "U405" H 3200 5317 50  0000 C CNN
+F 0 "U404" H 3200 5317 50  0000 C CNN
 F 1 "74HC04" H 3200 5226 50  0000 C CNN
 F 2 "" H 3200 5000 50  0001 C CNN
@@
 $EndComp
 $Comp
-L 74xx:74HC04 U405
+L 74xx:74HC04 U404
 U 3 1 60CDB507
 P 3200 6000
-F 0 "U405" H 3200 6317 50  0000 C CNN
+F 0 "U404" H 3200 6317 50  0000 C CNN
 F 1 "74HC04" H 3200 6226 50  0000 C CNN
 F 2 "" H 3200 6000 50  0001 C CNN
@@
 $EndComp
 $Comp
-L 74xx:74HC04 U405
+L 74xx:74HC04 U404
 U 4 1 60CDCB02
 P 8300 4750
-F 0 "U405" H 8300 5067 50  0000 C CNN
+F 0 "U404" H 8300 5067 50  0000 C CNN
 F 1 "74HC04" H 8300 4976 50  0000 C CNN
 F 2 "" H 8300 4750 50  0001 C CNN
@@
 $EndComp
 $Comp
-L 74xx:74HC04 U405
+L 74xx:74HC04 U404
 U 5 1 60CDEE27
 P 5000 5500
-F 0 "U405" H 5000 5817 50  0000 C CNN
+F 0 "U404" H 5000 5817 50  0000 C CNN
 F 1 "74HC04" H 5000 5726 50  0000 C CNN
 F 2 "" H 5000 5500 50  0001 C CNN
@@
 $EndComp
 $Comp
-L 74xx:74HC04 U405
+L 74xx:74HC04 U404
 U 6 1 60CE03D7
 P 8300 5850
-F 0 "U405" H 8300 6167 50  0000 C CNN
+F 0 "U404" H 8300 6167 50  0000 C CNN
 F 1 "74HC04" H 8300 6076 50  0000 C CNN
 F 2 "" H 8300 5850 50  0001 C CNN
@@
 $EndComp
 $Comp
-L 74xx:74HC04 U405
+L 74xx:74HC04 U404
 U 7 1 60CE187E
 P 9850 5250
-F 0 "U405" H 10080 5296 50  0000 L CNN
+F 0 "U404" H 10080 5296 50  0000 L CNN
 F 1 "74HC04" H 10080 5205 50  0000 L CNN
 F 2 "Package_SO:SOIC-14_3.9x8.7mm_P1.27mm" H 9850 5250 50  0001 C CNN
@@
 	2000 6100 2200 6100
 $Comp
-L power:GND #PWR0104
+L power:GND #PWR0414
 U 1 1 60D0672B
 P 800 7250
-F 0 "#PWR0104" H 800 7000 50  0001 C CNN
+F 0 "#PWR0414" H 800 7000 50  0001 C CNN
 F 1 "GND" V 805 7122 50  0000 R CNN
 F 2 "" H 800 7250 50  0001 C CNN
@@
 NoConn ~ 1650 7250
 $Comp
-L power:GND #PWR0105
+L power:GND #PWR0411
 U 1 1 60D10F62
 P 7550 5300
-F 0 "#PWR0105" H 7550 5050 50  0001 C CNN
+F 0 "#PWR0411" H 7550 5050 50  0001 C CNN
 F 1 "GND" V 7555 5172 50  0000 R CNN
 F 2 "" H 7550 5300 50  0001 C CNN
@@
 AR Path="/60D1B646" Ref="C?"  Part="1"
 AR Path="/60CA43D5/60D1B646" Ref="C?"  Part="1"
-AR Path="/60CB0F52/60D1B646" Ref="C402"  Part="1"
-F 0 "C402" V 2898 7150 50  0000 C CNN
+AR Path="/60CB0F52/60D1B646" Ref="C406"  Part="1"
+F 0 "C406" V 2898 7150 50  0000 C CNN
 F 1 "0.1uF" V 2989 7150 50  0000 C CNN
 F 2 "Capacitor_SMD:C_0603_1608Metric" H 3188 7000 50  0001 C CNN
@@
 AR Path="/60D1ED8C" Ref="C?"  Part="1"
 AR Path="/60CA43D5/60D1ED8C" Ref="C?"  Part="1"
-AR Path="/60CB0F52/60D1ED8C" Ref="C401"  Part="1"
-F 0 "C401" V 1798 2850 50  0000 C CNN
+AR Path="/60CB0F52/60D1ED8C" Ref="C403"  Part="1"
+F 0 "C403" V 1798 2850 50  0000 C CNN
 F 1 "0.1uF" V 1889 2850 50  0000 C CNN
 F 2 "Capacitor_SMD:C_0603_1608Metric" H 2088 2700 50  0001 C CNN
@@
 AR Path="/60D1FFA3" Ref="C?"  Part="1"
 AR Path="/60CA43D5/60D1FFA3" Ref="C?"  Part="1"
-AR Path="/60CB0F52/60D1FFA3" Ref="C403"  Part="1"
-F 0 "C403" V 4198 2750 50  0000 C CNN
+AR Path="/60CB0F52/60D1FFA3" Ref="C401"  Part="1"
+F 0 "C401" V 4198 2750 50  0000 C CNN
 F 1 "0.1uF" V 4289 2750 50  0000 C CNN
 F 2 "Capacitor_SMD:C_0603_1608Metric" H 4488 2600 50  0001 C CNN
@@
 	2050 2700 2050 2550
 $Comp
-L power:+5V #PWR0107
+L power:+5V #PWR0403
 U 1 1 60D273F3
 P 4550 2400
-F 0 "#PWR0107" H 4550 2250 50  0001 C CNN
+F 0 "#PWR0403" H 4550 2250 50  0001 C CNN
 F 1 "+5V" H 4565 2573 50  0000 C CNN
 F 2 "" H 4550 2400 50  0001 C CNN
@@
 	2050 2550 2200 2550
 $Comp
-L power:GND #PWR0106
+L power:GND #PWR0405
 U 1 1 60D311FD
 P 2200 2550
-F 0 "#PWR0106" H 2200 2300 50  0001 C CNN
+F 0 "#PWR0405" H 2200 2300 50  0001 C CNN
 F 1 "GND" H 2205 2377 50  0000 C CNN
 F 2 "" H 2200 2550 50  0001 C CNN
@@
 	2200 2550 2350 2550
 $Comp
-L power:GND #PWR0108
+L power:GND #PWR0406
 U 1 1 60D32007
 P 4550 3050
-F 0 "#PWR0108" H 4550 2800 50  0001 C CNN
+F 0 "#PWR0406" H 4550 2800 50  0001 C CNN
 F 1 "GND" H 4555 2877 50  0000 C CNN
 F 2 "" H 4550 3050 50  0001 C CNN
@@
 Connection ~ 4550 3050
 $Comp
-L power:+5V #PWR0109
+L power:+5V #PWR0409
 U 1 1 60D3A12D
 P 2250 3200
-F 0 "#PWR0109" H 2250 3050 50  0001 C CNN
+F 0 "#PWR0409" H 2250 3050 50  0001 C CNN
 F 1 "+5V" H 2265 3373 50  0000 C CNN
 F 2 "" H 2250 3200 50  0001 C CNN
@@
 Connection ~ 2250 3200
 $Comp
-L power:+5V #PWR0401
+L power:+5V #PWR0413
 U 1 1 60D3F3C4
 P 3150 6650
-F 0 "#PWR0401" H 3150 6500 50  0001 C CNN
+F 0 "#PWR0413" H 3150 6500 50  0001 C CNN
 F 1 "+5V" V 3165 6778 50  0000 L CNN
 F 2 "" H 3150 6650 50  0001 C CNN
@@
 $EndComp
 $Comp
-L power:GND #PWR0402
+L power:GND #PWR0415
 U 1 1 60D4000F
 P 3150 7650
-F 0 "#PWR0402" H 3150 7400 50  0001 C CNN
+F 0 "#PWR0415" H 3150 7400 50  0001 C CNN
 F 1 "GND" V 3155 7522 50  0000 R CNN
 F 2 "" H 3150 7650 50  0001 C CNN
@@
 Connection ~ 3150 6650
 $Comp
-L power:GND #PWR0408
+L power:GND #PWR0412
 U 1 1 60D48516
 P 10350 5900
-F 0 "#PWR0408" H 10350 5650 50  0001 C CNN
+F 0 "#PWR0412" H 10350 5650 50  0001 C CNN
 F 1 "GND" H 10355 5727 50  0000 C CNN
 F 2 "" H 10350 5900 50  0001 C CNN
@@
 	10700 4650 10700 5100
 $Comp
-L power:+5V #PWR0407
+L power:+5V #PWR0410
 U 1 1 60D50F40
 P 10250 4650
-F 0 "#PWR0407" H 10250 4500 50  0001 C CNN
+F 0 "#PWR0410" H 10250 4500 50  0001 C CNN
 F 1 "+5V" H 10265 4823 50  0000 C CNN
 F 2 "" H 10250 4650 50  0001 C CNN
@@
 	10250 4650 10700 4650
 $Comp
-L power:+5V #PWR0404
+L power:+5V #PWR0408
 U 1 1 60D51E1E
 P 7050 3100
-F 0 "#PWR0404" H 7050 2950 50  0001 C CNN
+F 0 "#PWR0408" H 7050 2950 50  0001 C CNN
 F 1 "+5V" H 7065 3273 50  0000 C CNN
 F 2 "" H 7050 3100 50  0001 C CNN
@@
 $EndComp
 $Comp
-L power:GND #PWR0403
+L power:GND #PWR0404
 U 1 1 60D52CD0
 P 7000 2450
-F 0 "#PWR0403" H 7000 2200 50  0001 C CNN
+F 0 "#PWR0404" H 7000 2200 50  0001 C CNN
 F 1 "GND" H 7005 2277 50  0000 C CNN
 F 2 "" H 7000 2450 50  0001 C CNN
@@
 Connection ~ 7050 3100
 $Comp
-L power:+5V #PWR0405
+L power:+5V #PWR0401
 U 1 1 60C9A9B2
 P 9900 1900
-F 0 "#PWR0405" H 9900 1750 50  0001 C CNN
+F 0 "#PWR0401" H 9900 1750 50  0001 C CNN
 F 1 "+5V" H 9915 2073 50  0000 C CNN
 F 2 "" H 9900 1900 50  0001 C CNN
@@
 AR Path="/60B094D9/60C9A9B9" Ref="R?"  Part="1"
 AR Path="/60B13096/60C9A9B9" Ref="R?"  Part="1"
-AR Path="/60CB0F52/60C9A9B9" Ref="R402"  Part="1"
-F 0 "R402" H 9970 2196 50  0000 L CNN
+AR Path="/60CB0F52/60C9A9B9" Ref="R401"  Part="1"
+F 0 "R401" H 9970 2196 50  0000 L CNN
 F 1 "1k" H 9970 2105 50  0000 L CNN
 F 2 "Resistor_SMD:R_0603_1608Metric" V 9830 2150 50  0001 C CNN
@@
 AR Path="/60B094D9/60C9A9C0" Ref="R?"  Part="1"
 AR Path="/60B13096/60C9A9C0" Ref="R?"  Part="1"
-AR Path="/60CB0F52/60C9A9C0" Ref="R401"  Part="1"
-F 0 "R401" H 9570 2846 50  0000 L CNN
+AR Path="/60CB0F52/60C9A9C0" Ref="R402"  Part="1"
+F 0 "R402" H 9570 2846 50  0000 L CNN
 F 1 "180k" H 9570 2755 50  0000 L CNN
 F 2 "Resistor_SMD:R_0603_1608Metric" V 9430 2800 50  0001 C CNN
@@
 AR Path="/60B094D9/60C9A9C7" Ref="C?"  Part="1"
 AR Path="/60B13096/60C9A9C7" Ref="C?"  Part="1"
-AR Path="/60CB0F52/60C9A9C7" Ref="C406"  Part="1"
-F 0 "C406" H 10415 2846 50  0000 L CNN
+AR Path="/60CB0F52/60C9A9C7" Ref="C402"  Part="1"
+F 0 "C402" H 10415 2846 50  0000 L CNN
 F 1 "10u" H 10415 2755 50  0000 L CNN
 F 2 "Capacitor_SMD:C_0603_1608Metric" H 10338 2650 50  0001 C CNN
@@
 $EndComp
 $Comp
-L power:GND #PWR0406
+L power:GND #PWR0407
 U 1 1 60C9A9CD
 P 9900 3050
-F 0 "#PWR0406" H 9900 2800 50  0001 C CNN
+F 0 "#PWR0407" H 9900 2800 50  0001 C CNN
 F 1 "GND" H 9905 2877 50  0000 C CNN
 F 2 "" H 9900 3050 50  0001 C CNN

Commit message: Fix output enable, and do some routing
Connections:
- net +5V: no longer U402.13 (~G)
- net GND: now also U402.13 (~G)
Changed lines of the file:
@@
 	0    -1   1    0
-$EndComp
-$Comp
-L power:+5V #PWR0402
-U 1 1 60CBA05E
-P 4900 2000
-F 0 "#PWR0402" H 4900 1850 50  0001 C CNN
-F 1 "+5V" H 4915 2173 50  0000 C CNN
-F 2 "" H 4900 2000 50  0001 C CNN
-F 3 "" H 4900 2000 50  0001 C CNN
-	1    4900 2000
-	1    0    0    -1
 $EndComp
 Wire Wire Line
@@
 	9200 2300 9500 2300
 Connection ~ 9500 2300
+$Comp
+L power:GND #PWR?
+U 1 1 60CE1890
+P 4900 2000
+F 0 "#PWR?" H 4900 1750 50  0001 C CNN
+F 1 "GND" H 4905 1827 50  0000 C CNN
+F 2 "" H 4900 2000 50  0001 C CNN
+F 3 "" H 4900 2000 50  0001 C CNN
+	1    4900 2000
+	-1   0    0    1
+$EndComp
 $EndSCHEMATC
