File: SPI LED 8x8/LED8x8.sch (KiCad schematic (older format))
At the start: 19 parts, among them J101 Conn_01x05_Male, Q101 2N3904, U101 74HCT125, U102 74HC138, U103 4024

Commit message: Updating values
Parts:
- C102, C103, C104: value C -> 0.1uF
Changed lines of the file:
@@
 P 5600 1600
 F 0 "C103" H 5485 1554 50  0000 R CNN
-F 1 "C" H 5485 1645 50  0000 R CNN
+F 1 "0.1uF" H 5485 1645 50  0000 R CNN
 F 2 "Capacitor_THT:C_Disc_D4.7mm_W2.5mm_P5.00mm" H 5638 1450 50  0001 C CNN
 F 3 "~" H 5600 1600 50  0001 C CNN
@@
 P 1000 6250
 F 0 "C104" H 885 6204 50  0000 R CNN
-F 1 "C" H 885 6295 50  0000 R CNN
+F 1 "0.1uF" H 885 6295 50  0000 R CNN
 F 2 "Capacitor_THT:C_Disc_D4.7mm_W2.5mm_P5.00mm" H 1038 6100 50  0001 C CNN
 F 3 "~" H 1000 6250 50  0001 C CNN
@@
 AR Path="/60E8CBBD" Ref="C102"  Part="1"
 F 0 "C102" H 7135 1504 50  0000 R CNN
-F 1 "C" H 7135 1595 50  0000 R CNN
+F 1 "0.1uF" H 7135 1595 50  0000 R CNN
 F 2 "Capacitor_THT:C_Disc_D4.3mm_W1.9mm_P5.00mm" H 7288 1400 50  0001 C CNN
 F 3 "~" H 7250 1550 50  0001 C CNN
