File: SPI LED 8x8/file602AD596.sch (KiCad schematic (older format))
At the start: 16 parts, among them U501 74HC574, U502 74HC574, U503 74HC574, U504 74HC574, U505 74HC574, U506 74HC574, U507 74HC574, U508 74HC574

Commit message: More values
Parts:
- C501, C502, C503, C504, C505, C506, C507, C508: value C -> 0.1uF
Changed lines of the file:
@@
 P 2800 900
 F 0 "C501" H 2685 854 50  0000 R CNN
-F 1 "C" H 2685 945 50  0000 R CNN
+F 1 "0.1uF" H 2685 945 50  0000 R CNN
 F 2 "Capacitor_THT:C_Disc_D4.3mm_W1.9mm_P5.00mm" H 2838 750 50  0001 C CNN
 F 3 "~" H 2800 900 50  0001 C CNN
@@
 P 4500 900
 F 0 "C503" H 4385 854 50  0000 R CNN
-F 1 "C" H 4385 945 50  0000 R CNN
+F 1 "0.1uF" H 4385 945 50  0000 R CNN
 F 2 "Capacitor_THT:C_Disc_D4.3mm_W1.9mm_P5.00mm" H 4538 750 50  0001 C CNN
 F 3 "~" H 4500 900 50  0001 C CNN
@@
 P 6200 900
 F 0 "C505" H 6085 854 50  0000 R CNN
-F 1 "C" H 6085 945 50  0000 R CNN
+F 1 "0.1uF" H 6085 945 50  0000 R CNN
 F 2 "Capacitor_THT:C_Disc_D4.3mm_W1.9mm_P5.00mm" H 6238 750 50  0001 C CNN
 F 3 "~" H 6200 900 50  0001 C CNN
@@
 P 7900 900
 F 0 "C507" H 7785 854 50  0000 R CNN
-F 1 "C" H 7785 945 50  0000 R CNN
+F 1 "0.1uF" H 7785 945 50  0000 R CNN
 F 2 "Capacitor_THT:C_Disc_D4.3mm_W1.9mm_P5.00mm" H 7938 750 50  0001 C CNN
 F 3 "~" H 7900 900 50  0001 C CNN
@@
 P 2800 3950
 F 0 "C502" H 2685 3904 50  0000 R CNN
-F 1 "C" H 2685 3995 50  0000 R CNN
+F 1 "0.1uF" H 2685 3995 50  0000 R CNN
 F 2 "Capacitor_THT:C_Disc_D4.3mm_W1.9mm_P5.00mm" H 2838 3800 50  0001 C CNN
 F 3 "~" H 2800 3950 50  0001 C CNN
@@
 P 4500 3950
 F 0 "C504" H 4385 3904 50  0000 R CNN
-F 1 "C" H 4385 3995 50  0000 R CNN
+F 1 "0.1uF" H 4385 3995 50  0000 R CNN
 F 2 "Capacitor_THT:C_Disc_D4.3mm_W1.9mm_P5.00mm" H 4538 3800 50  0001 C CNN
 F 3 "~" H 4500 3950 50  0001 C CNN
@@
 P 6200 3950
 F 0 "C506" H 6085 3904 50  0000 R CNN
-F 1 "C" H 6085 3995 50  0000 R CNN
+F 1 "0.1uF" H 6085 3995 50  0000 R CNN
 F 2 "Capacitor_THT:C_Disc_D4.3mm_W1.9mm_P5.00mm" H 6238 3800 50  0001 C CNN
 F 3 "~" H 6200 3950 50  0001 C CNN
@@
 P 7900 3950
 F 0 "C508" H 7785 3904 50  0000 R CNN
-F 1 "C" H 7785 3995 50  0000 R CNN
+F 1 "0.1uF" H 7785 3995 50  0000 R CNN
 F 2 "Capacitor_THT:C_Disc_D4.3mm_W1.9mm_P5.00mm" H 7938 3800 50  0001 C CNN
 F 3 "~" H 7900 3950 50  0001 C CNN
