File: SPI LED 8x8/file6024758F.sch (KiCad schematic (older format))
At the start: 104 parts, among them Q401 2N3906, Q402 2N3906, Q403 2N3906, Q404 2N3906, Q405 2N3906, Q406 2N3906, Q407 2N3906, Q408 2N3906, Q409 2N3904, Q410 2N3904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

Commit message: More values
Parts:
- R401, R402, R403, R404, R406, R407, R408: value R -> 4k7
Changed lines of the file:
@@
 P 2350 4300
 F 0 "R408" H 2420 4346 50  0000 L CNN
-F 1 "R" H 2420 4255 50  0000 L CNN
+F 1 "4k7" H 2420 4255 50  0000 L CNN
 F 2 "Resistor_THT:R_Axial_DIN0207_L6.3mm_D2.5mm_P7.62mm_Horizontal" V 2280 4300 50  0001 C CNN
 F 3 "~" H 2350 4300 50  0001 C CNN
@@
 P 2350 3800
 F 0 "R407" H 2420 3846 50  0000 L CNN
-F 1 "R" H 2420 3755 50  0000 L CNN
+F 1 "4k7" H 2420 3755 50  0000 L CNN
 F 2 "Resistor_THT:R_Axial_DIN0207_L6.3mm_D2.5mm_P7.62mm_Horizontal" V 2280 3800 50  0001 C CNN
 F 3 "~" H 2350 3800 50  0001 C CNN
@@
 P 2350 3300
 F 0 "R406" H 2420 3346 50  0000 L CNN
-F 1 "R" H 2420 3255 50  0000 L CNN
+F 1 "4k7" H 2420 3255 50  0000 L CNN
 F 2 "Resistor_THT:R_Axial_DIN0207_L6.3mm_D2.5mm_P7.62mm_Horizontal" V 2280 3300 50  0001 C CNN
 F 3 "~" H 2350 3300 50  0001 C CNN
@@
 P 2350 2300
 F 0 "R404" H 2420 2346 50  0000 L CNN
-F 1 "R" H 2420 2255 50  0000 L CNN
+F 1 "4k7" H 2420 2255 50  0000 L CNN
 F 2 "Resistor_THT:R_Axial_DIN0207_L6.3mm_D2.5mm_P7.62mm_Horizontal" V 2280 2300 50  0001 C CNN
 F 3 "~" H 2350 2300 50  0001 C CNN
@@
 P 2350 1800
 F 0 "R403" H 2420 1846 50  0000 L CNN
-F 1 "R" H 2420 1755 50  0000 L CNN
+F 1 "4k7" H 2420 1755 50  0000 L CNN
 F 2 "Resistor_THT:R_Axial_DIN0207_L6.3mm_D2.5mm_P7.62mm_Horizontal" V 2280 1800 50  0001 C CNN
 F 3 "~" H 2350 1800 50  0001 C CNN
@@
 P 2350 1300
 F 0 "R402" H 2420 1346 50  0000 L CNN
-F 1 "R" H 2420 1255 50  0000 L CNN
+F 1 "4k7" H 2420 1255 50  0000 L CNN
 F 2 "Resistor_THT:R_Axial_DIN0207_L6.3mm_D2.5mm_P7.62mm_Horizontal" V 2280 1300 50  0001 C CNN
 F 3 "~" H 2350 1300 50  0001 C CNN
@@
 P 2350 800
 F 0 "R401" H 2420 846 50  0000 L CNN
-F 1 "R" H 2420 755 50  0000 L CNN
+F 1 "4k7" H 2420 755 50  0000 L CNN
 F 2 "Resistor_THT:R_Axial_DIN0207_L6.3mm_D2.5mm_P7.62mm_Horizontal" V 2280 800 50  0001 C CNN
 F 3 "~" H 2350 800 50  0001 C CNN

Commit message: Filling in resistors
Parts:
- R409, R410, R411, R412, R413, R414, R415, R416: value R -> 1k
- R417, R418, R419, R420, R421, R422, R423, R424: value R -> 10k
Changed lines of the file:
@@
 P 3500 5150
 F 0 "R409" H 3570 5196 50  0000 L CNN
-F 1 "R" H 3570 5105 50  0000 L CNN
+F 1 "1k" H 3570 5105 50  0000 L CNN
 F 2 "Resistor_THT:R_Axial_DIN0207_L6.3mm_D2.5mm_P7.62mm_Horizontal" V 3430 5150 50  0001 C CNN
 F 3 "~" H 3500 5150 50  0001 C CNN
@@
 P 4500 5150
 F 0 "R410" H 4570 5196 50  0000 L CNN
-F 1 "R" H 4570 5105 50  0000 L CNN
+F 1 "1k" H 4570 5105 50  0000 L CNN
 F 2 "Resistor_THT:R_Axial_DIN0207_L6.3mm_D2.5mm_P7.62mm_Horizontal" V 4430 5150 50  0001 C CNN
 F 3 "~" H 4500 5150 50  0001 C CNN
@@
 P 5500 5150
 F 0 "R411" H 5570 5196 50  0000 L CNN
-F 1 "R" H 5570 5105 50  0000 L CNN
+F 1 "1k" H 5570 5105 50  0000 L CNN
 F 2 "Resistor_THT:R_Axial_DIN0207_L6.3mm_D2.5mm_P7.62mm_Horizontal" V 5430 5150 50  0001 C CNN
 F 3 "~" H 5500 5150 50  0001 C CNN
@@
 P 6500 5150
 F 0 "R412" H 6570 5196 50  0000 L CNN
-F 1 "R" H 6570 5105 50  0000 L CNN
+F 1 "1k" H 6570 5105 50  0000 L CNN
 F 2 "Resistor_THT:R_Axial_DIN0207_L6.3mm_D2.5mm_P7.62mm_Horizontal" V 6430 5150 50  0001 C CNN
 F 3 "~" H 6500 5150 50  0001 C CNN
@@
 P 7500 5150
 F 0 "R413" H 7570 5196 50  0000 L CNN
-F 1 "R" H 7570 5105 50  0000 L CNN
+F 1 "1k" H 7570 5105 50  0000 L CNN
 F 2 "Resistor_THT:R_Axial_DIN0207_L6.3mm_D2.5mm_P7.62mm_Horizontal" V 7430 5150 50  0001 C CNN
 F 3 "~" H 7500 5150 50  0001 C CNN
@@
 P 8500 5150
 F 0 "R414" H 8570 5196 50  0000 L CNN
-F 1 "R" H 8570 5105 50  0000 L CNN
+F 1 "1k" H 8570 5105 50  0000 L CNN
 F 2 "Resistor_THT:R_Axial_DIN0207_L6.3mm_D2.5mm_P7.62mm_Horizontal" V 8430 5150 50  0001 C CNN
 F 3 "~" H 8500 5150 50  0001 C CNN
@@
 P 9500 5150
 F 0 "R415" H 9570 5196 50  0000 L CNN
-F 1 "R" H 9570 5105 50  0000 L CNN
+F 1 "1k" H 9570 5105 50  0000 L CNN
 F 2 "Resistor_THT:R_Axial_DIN0207_L6.3mm_D2.5mm_P7.62mm_Horizontal" V 9430 5150 50  0001 C CNN
 F 3 "~" H 9500 5150 50  0001 C CNN
@@
 P 10500 5150
 F 0 "R416" H 10570 5196 50  0000 L CNN
-F 1 "R" H 10570 5105 50  0000 L CNN
+F 1 "1k" H 10570 5105 50  0000 L CNN
 F 2 "Resistor_THT:R_Axial_DIN0207_L6.3mm_D2.5mm_P7.62mm_Horizontal" V 10430 5150 50  0001 C CNN
 F 3 "~" H 10500 5150 50  0001 C CNN
@@
 P 3000 6000
 F 0 "R417" H 3070 6046 50  0000 L CNN
-F 1 "R" H 3070 5955 50  0000 L CNN
+F 1 "10k" H 3070 5955 50  0000 L CNN
 F 2 "Resistor_THT:R_Axial_DIN0207_L6.3mm_D2.5mm_P7.62mm_Horizontal" V 2930 6000 50  0001 C CNN
 F 3 "~" H 3000 6000 50  0001 C CNN
@@
 P 4000 6000
 F 0 "R418" H 4070 6046 50  0000 L CNN
-F 1 "R" H 4070 5955 50  0000 L CNN
+F 1 "10k" H 4070 5955 50  0000 L CNN
 F 2 "Resistor_THT:R_Axial_DIN0207_L6.3mm_D2.5mm_P7.62mm_Horizontal" V 3930 6000 50  0001 C CNN
 F 3 "~" H 4000 6000 50  0001 C CNN
@@
 P 5000 6000
 F 0 "R419" H 5070 6046 50  0000 L CNN
-F 1 "R" H 5070 5955 50  0000 L CNN
+F 1 "10k" H 5070 5955 50  0000 L CNN
 F 2 "Resistor_THT:R_Axial_DIN0207_L6.3mm_D2.5mm_P7.62mm_Horizontal" V 4930 6000 50  0001 C CNN
 F 3 "~" H 5000 6000 50  0001 C CNN
@@
 P 6000 6000
 F 0 "R420" H 6070 6046 50  0000 L CNN
-F 1 "R" H 6070 5955 50  0000 L CNN
+F 1 "10k" H 6070 5955 50  0000 L CNN
 F 2 "Resistor_THT:R_Axial_DIN0207_L6.3mm_D2.5mm_P7.62mm_Horizontal" V 5930 6000 50  0001 C CNN
 F 3 "~" H 6000 6000 50  0001 C CNN
@@
 P 7000 6000
 F 0 "R421" H 7070 6046 50  0000 L CNN
-F 1 "R" H 7070 5955 50  0000 L CNN
+F 1 "10k" H 7070 5955 50  0000 L CNN
 F 2 "Resistor_THT:R_Axial_DIN0207_L6.3mm_D2.5mm_P7.62mm_Horizontal" V 6930 6000 50  0001 C CNN
 F 3 "~" H 7000 6000 50  0001 C CNN
@@
 P 8000 6000
 F 0 "R422" H 8070 6046 50  0000 L CNN
-F 1 "R" H 8070 5955 50  0000 L CNN
+F 1 "10k" H 8070 5955 50  0000 L CNN
 F 2 "Resistor_THT:R_Axial_DIN0207_L6.3mm_D2.5mm_P7.62mm_Horizontal" V 7930 6000 50  0001 C CNN
 F 3 "~" H 8000 6000 50  0001 C CNN
@@
 P 9000 6000
 F 0 "R423" H 9070 6046 50  0000 L CNN
-F 1 "R" H 9070 5955 50  0000 L CNN
+F 1 "10k" H 9070 5955 50  0000 L CNN
 F 2 "Resistor_THT:R_Axial_DIN0207_L6.3mm_D2.5mm_P7.62mm_Horizontal" V 8930 6000 50  0001 C CNN
 F 3 "~" H 9000 6000 50  0001 C CNN
@@
 P 10000 6000
 F 0 "R424" H 10070 6046 50  0000 L CNN
-F 1 "R" H 10070 5955 50  0000 L CNN
+F 1 "10k" H 10070 5955 50  0000 L CNN
 F 2 "Resistor_THT:R_Axial_DIN0207_L6.3mm_D2.5mm_P7.62mm_Horizontal" V 9930 6000 50  0001 C CNN
 F 3 "~" H 10000 6000 50  0001 C CNN

Commit message: Missed some
Parts:
- R405: value R -> 4k7
Changed lines of the file:
@@
 P 2350 2800
 F 0 "R405" H 2420 2846 50  0000 L CNN
-F 1 "R" H 2420 2755 50  0000 L CNN
+F 1 "4k7" H 2420 2755 50  0000 L CNN
 F 2 "Resistor_THT:R_Axial_DIN0207_L6.3mm_D2.5mm_P7.62mm_Horizontal" V 2280 2800 50  0001 C CNN
 F 3 "~" H 2350 2800 50  0001 C CNN
