File: SPI LED 8x8/file60630695.sch (KiCad schematic (older format))
At the start: 4 parts, among them U301 74HC164, U302 74HC164

Commit message: Four more
Parts:
- C301, C302: value 0.1u -> 0.1uF
Changed lines of the file:
@@
 P 2050 3750
 F 0 "C302" H 2165 3796 50  0000 L CNN
-F 1 "0.1u" H 2165 3705 50  0000 L CNN
+F 1 "0.1uF" H 2165 3705 50  0000 L CNN
 F 2 "Capacitor_THT:C_Disc_D4.3mm_W1.9mm_P5.00mm" H 2088 3600 50  0001 C CNN
 F 3 "~" H 2050 3750 50  0001 C CNN
@@
 P 2100 1650
 F 0 "C301" H 2215 1696 50  0000 L CNN
-F 1 "0.1u" H 2215 1605 50  0000 L CNN
+F 1 "0.1uF" H 2215 1605 50  0000 L CNN
 F 2 "Capacitor_THT:C_Disc_D4.3mm_W1.9mm_P5.00mm" H 2138 1500 50  0001 C CNN
 F 3 "~" H 2100 1650 50  0001 C CNN
