File: 3V3 to 5V Level Shifter/3V3 to 5V Level Shifter.kicad_pcb (KiCad board)
At the start: 2 copper layers, 50.8 x 63.5 mm, 17 parts, among them J1001 Conn_01x02_Male, J1002 Conn_01x04_Male, J1003 Conn_01x04_Male, J1004 Conn_01x04_Male, J1005 Conn_01x04_Male, U1001 74LVC125, U1002 74LVC125

Commit message: Finishing design
Parts:
- added J1006: Conn_01x02_Male, Connector_PinHeader_2.54mm:PinHeader_1x02_P2.54mm_Vertical, F.Cu at (100.3, 91.4)
Routing:
- net Net-(J1002-Pad4): track 0.00 -> 47.7 mm, vias 0 -> 1
- net Net-(J1004-Pad4): track 0.00 -> 47.7 mm, vias 0 -> 1
- net Net-(J1004-Pad3): track 0.00 -> 43.0 mm
- net Net-(J1002-Pad3): track 0.00 -> 43.0 mm
- net Net-(J1005-Pad2): track 0.00 -> 32.8 mm
- net Net-(J1003-Pad2): track 0.00 -> 32.8 mm
- net Net-(J1005-Pad1): track 0.00 -> 24.3 mm
- net Net-(J1003-Pad1): track 0.00 -> 24.3 mm
- net Net-(J1005-Pad3): track 0.00 -> 22.1 mm
- net Net-(J1003-Pad3): track 0.00 -> 22.1 mm
- net Net-(J1004-Pad2): track 0.00 -> 16.7 mm
- net Net-(J1002-Pad2): track 0.00 -> 16.7 mm
- net Net-(J1003-Pad4): track 0.00 -> 14.5 mm
- net Net-(J1005-Pad4): track 0.00 -> 14.5 mm
- net Net-(J1002-Pad1): track 0.00 -> 12.3 mm
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- added copper zone on B.Cu, net +5V
- added copper zone on F.Cu, net GND
Other:
- board size 50.8 x 63.5 mm -> 43.2 x 62.2 mm
- board text added: "RGE2021"

Commit message: Correct IC name
Parts:
- U1001, U1002: value 74LVC125 -> 74AHCT125
