File: Shift Register Tutorial/file61B7DA08.sch (KiCad schematic (older format))
At the start: 7 parts, among them Q401 2N3904, SW401 SW_Push

Commit message: Disconnect indicator LEDs
Connections:
- net ~RESET: no longer Q401.2 (B)
Changed lines of the file:
@@
 	1    0    0    -1
 $EndComp
-Wire Wire Line
-	2900 2850 3750 2850
 $Comp
 L power:GND #PWR?
@@
 Wire Wire Line
 	2500 1450 2500 1650
-Wire Wire Line
-	2500 2550 2900 2550
 Connection ~ 2500 2550
 Wire Wire Line
 	2500 2550 2500 2650
-Wire Wire Line
-	2900 2850 2900 2550
-Connection ~ 2900 2550
-Wire Wire Line
-	2900 2550 3100 2550
 Wire Wire Line
 	1800 2050 2500 2050
@@
 	0    1    1    0
 $EndComp
+Wire Wire Line
+	2500 2550 3100 2550
 $EndSCHEMATC

Commit message: Rerouting board
Parts:
- removed D401: LED, LED_THT:LED_D5.0mm, symbol Device:LED
- removed Q401: 2N3904, Package_TO_SOT_THT:TO-92_Inline_Wide, symbol Transistor_BJT:2N3904
- removed R403: 2k2, Resistor_THT:R_Axial_DIN0207_L6.3mm_D2.5mm_P7.62mm_Horizontal, symbol Device:R
- C401: value 1u -> 10u
Changed lines of the file:
@@
 AR Path="/61B7DA09/61B80A0C" Ref="C401"  Part="1"
 F 0 "C401" H 2618 2846 50  0000 L CNN
-F 1 "1u" H 2618 2755 50  0000 L CNN
+F 1 "10u" H 2618 2755 50  0000 L CNN
 F 2 "Capacitor_THT:CP_Radial_D4.0mm_P2.00mm" H 2538 2650 50  0001 C CNN
 F 3 "~" H 2500 2800 50  0001 C CNN
@@
 Text HLabel 3100 2550 2    50   Output ~ 0
 ~RESET
-$Comp
-L Transistor_BJT:2N3904 Q?
-U 1 1 61B80A34
-P 3950 2850
-AR Path="/61B52EB5/61B80A34" Ref="Q?"  Part="1"
-AR Path="/61B7DA09/61B80A34" Ref="Q401"  Part="1"
-F 0 "Q401" H 4140 2896 50  0000 L CNN
-F 1 "2N3904" H 4140 2805 50  0000 L CNN
-F 2 "Package_TO_SOT_THT:TO-92_Inline_Wide" H 4150 2775 50  0001 L CIN
-F 3 "https://www.onsemi.com/pub/Collateral/2N3903-D.PDF" H 3950 2850 50  0001 L CNN
-	1    3950 2850
-	1    0    0    -1
-$EndComp
-$Comp
-L power:GND #PWR?
-U 1 1 61B80A3E
-P 4050 3400
-AR Path="/61B52EB5/61B80A3E" Ref="#PWR?"  Part="1"
-AR Path="/61B7DA09/61B80A3E" Ref="#PWR0404"  Part="1"
-F 0 "#PWR0404" H 4050 3150 50  0001 C CNN
-F 1 "GND" H 4055 3227 50  0000 C CNN
-F 2 "" H 4050 3400 50  0001 C CNN
-F 3 "" H 4050 3400 50  0001 C CNN
-	1    4050 3400
-	1    0    0    -1
-$EndComp
-Wire Wire Line
-	4050 3050 4050 3400
-$Comp
-L Device:R R?
-U 1 1 61B80A45
-P 4050 2300
-AR Path="/61B52EB5/61B80A45" Ref="R?"  Part="1"
-AR Path="/61B7DA09/61B80A45" Ref="R403"  Part="1"
-F 0 "R403" H 4120 2346 50  0000 L CNN
-F 1 "2k2" H 4120 2255 50  0000 L CNN
-F 2 "Resistor_THT:R_Axial_DIN0207_L6.3mm_D2.5mm_P7.62mm_Horizontal" V 3980 2300 50  0001 C CNN
-F 3 "~" H 4050 2300 50  0001 C CNN
-	1    4050 2300
-	1    0    0    -1
-$EndComp
-$Comp
-L Device:LED D?
-U 1 1 61B80A4B
-P 4050 1800
-AR Path="/61B52EB5/61B80A4B" Ref="D?"  Part="1"
-AR Path="/61B7DA09/61B80A4B" Ref="D401"  Part="1"
-F 0 "D401" V 4089 1682 50  0000 R CNN
-F 1 "LED" V 3998 1682 50  0000 R CNN
-F 2 "LED_THT:LED_D5.0mm" H 4050 1800 50  0001 C CNN
-F 3 "~" H 4050 1800 50  0001 C CNN
-	1    4050 1800
-	0    -1   -1   0
-$EndComp
-$Comp
-L power:+5V #PWR?
-U 1 1 61B80A51
-P 4050 1400
-AR Path="/61B52EB5/61B80A51" Ref="#PWR?"  Part="1"
-AR Path="/61B7DA09/61B80A51" Ref="#PWR0403"  Part="1"
-F 0 "#PWR0403" H 4050 1250 50  0001 C CNN
-F 1 "+5V" H 4065 1573 50  0000 C CNN
-F 2 "" H 4050 1400 50  0001 C CNN
-F 3 "" H 4050 1400 50  0001 C CNN
-	1    4050 1400
-	1    0    0    -1
-$EndComp
-Wire Wire Line
-	4050 1400 4050 1650
-Wire Wire Line
-	4050 1950 4050 2150
-Wire Wire Line
-	4050 2450 4050 2650
 Wire Wire Line
 	2500 1950 2500 2050

Commit message: Removing old things
Parts:
- removed C401: 10u, Capacitor_THT:CP_Radial_D4.0mm_P2.00mm, symbol Device:CP
- removed R401: 10k, Resistor_THT:R_Axial_DIN0207_L6.3mm_D2.5mm_P7.62mm_Horizontal, symbol Device:R
- renumbered R402 to R401
Connections:
- net +5V: now also R401.1
- net GND: now also SW401.1; no longer SW401.2
- net ~RESET: now also SW401.2
Other:
- moved on the sheet: SW401
Changed lines of the file:
@@
-$Comp
-L Device:R R?
-U 1 1 61B80A00
-P 2500 1800
-AR Path="/61B52EB5/61B80A00" Ref="R?"  Part="1"
-AR Path="/61B7DA09/61B80A00" Ref="R401"  Part="1"
-F 0 "R401" H 2570 1846 50  0000 L CNN
-F 1 "10k" H 2570 1755 50  0000 L CNN
-F 2 "Resistor_THT:R_Axial_DIN0207_L6.3mm_D2.5mm_P7.62mm_Horizontal" V 2430 1800 50  0001 C CNN
-F 3 "~" H 2500 1800 50  0001 C CNN
-	1    2500 1800
-	1    0    0    -1
-$EndComp
 $Comp
 L Device:R R?
@@
 P 2500 2300
 AR Path="/61B52EB5/61B80A06" Ref="R?"  Part="1"
-AR Path="/61B7DA09/61B80A06" Ref="R402"  Part="1"
-F 0 "R402" H 2570 2346 50  0000 L CNN
+AR Path="/61B7DA09/61B80A06" Ref="R401"  Part="1"
+F 0 "R401" H 2570 2346 50  0000 L CNN
 F 1 "22k" H 2570 2255 50  0000 L CNN
 F 2 "Resistor_THT:R_Axial_DIN0207_L6.3mm_D2.5mm_P7.62mm_Horizontal" V 2430 2300 50  0001 C CNN
@@
 $EndComp
 $Comp
-L Device:CP C?
-U 1 1 61B80A0C
-P 2500 2800
-AR Path="/61B52EB5/61B80A0C" Ref="C?"  Part="1"
-AR Path="/61B7DA09/61B80A0C" Ref="C401"  Part="1"
-F 0 "C401" H 2618 2846 50  0000 L CNN
-F 1 "10u" H 2618 2755 50  0000 L CNN
-F 2 "Capacitor_THT:CP_Radial_D4.0mm_P2.00mm" H 2538 2650 50  0001 C CNN
-F 3 "~" H 2500 2800 50  0001 C CNN
-	1    2500 2800
-	1    0    0    -1
-$EndComp
-$Comp
 L power:+5V #PWR?
 U 1 1 61B80A12
-P 2500 1450
+P 2500 1900
 AR Path="/61B52EB5/61B80A12" Ref="#PWR?"  Part="1"
 AR Path="/61B7DA09/61B80A12" Ref="#PWR0401"  Part="1"
-F 0 "#PWR0401" H 2500 1300 50  0001 C CNN
-F 1 "+5V" H 2515 1623 50  0000 C CNN
-F 2 "" H 2500 1450 50  0001 C CNN
-F 3 "" H 2500 1450 50  0001 C CNN
-	1    2500 1450
+F 0 "#PWR0401" H 2500 1750 50  0001 C CNN
+F 1 "+5V" H 2515 2073 50  0000 C CNN
+F 2 "" H 2500 1900 50  0001 C CNN
+F 3 "" H 2500 1900 50  0001 C CNN
+	1    2500 1900
 	1    0    0    -1
 $EndComp
@@
 L power:GND #PWR?
 U 1 1 61B80A18
-P 2500 3100
+P 2500 3300
 AR Path="/61B52EB5/61B80A18" Ref="#PWR?"  Part="1"
 AR Path="/61B7DA09/61B80A18" Ref="#PWR0402"  Part="1"
-F 0 "#PWR0402" H 2500 2850 50  0001 C CNN
-F 1 "GND" H 2505 2927 50  0000 C CNN
-F 2 "" H 2500 3100 50  0001 C CNN
-F 3 "" H 2500 3100 50  0001 C CNN
-	1    2500 3100
+F 0 "#PWR0402" H 2500 3050 50  0001 C CNN
+F 1 "GND" H 2505 3127 50  0000 C CNN
+F 2 "" H 2500 3300 50  0001 C CNN
+F 3 "" H 2500 3300 50  0001 C CNN
+	1    2500 3300
 	1    0    0    -1
 $EndComp
-Wire Wire Line
-	2500 2950 2500 3000
 Text HLabel 3100 2550 2    50   Output ~ 0
 ~RESET
 Wire Wire Line
-	2500 1950 2500 2050
-Wire Wire Line
 	2500 2450 2500 2550
-Wire Wire Line
-	2500 1450 2500 1650
 Connection ~ 2500 2550
-Wire Wire Line
-	2500 2550 2500 2650
-Wire Wire Line
-	1800 2050 2500 2050
-Connection ~ 2500 2050
-Wire Wire Line
-	2500 2050 2500 2150
-Wire Wire Line
-	1800 2700 1800 3000
-Wire Wire Line
-	1800 3000 2500 3000
-Connection ~ 2500 3000
-Wire Wire Line
-	2500 3000 2500 3100
-Wire Wire Line
-	1800 2300 1800 2050
 $Comp
 L Switch:SW_Push SW?
 U 1 1 61B80A22
-P 1800 2500
+P 2500 2950
 AR Path="/61B52EB5/61B80A22" Ref="SW?"  Part="1"
 AR Path="/61B7DA09/61B80A22" Ref="SW401"  Part="1"
-F 0 "SW401" V 1754 2648 50  0000 L CNN
-F 1 "SW_Push" V 1845 2648 50  0000 L CNN
-F 2 "Button_Switch_THT:SW_PUSH_6mm_H4.3mm" H 1800 2700 50  0001 C CNN
-F 3 "~" H 1800 2700 50  0001 C CNN
-	1    1800 2500
-	0    1    1    0
+F 0 "SW401" V 2454 3098 50  0000 L CNN
+F 1 "SW_Push" V 2545 3098 50  0000 L CNN
+F 2 "Button_Switch_THT:SW_PUSH_6mm_H4.3mm" H 2500 3150 50  0001 C CNN
+F 3 "~" H 2500 3150 50  0001 C CNN
+	1    2500 2950
+	0    -1   -1   0
 $EndComp
 Wire Wire Line
 	2500 2550 3100 2550
+Wire Wire Line
+	2500 2550 2500 2750
+Wire Wire Line
+	2500 3150 2500 3300
+Wire Wire Line
+	2500 2150 2500 1900
 $EndSCHEMATC

Commit message: Working circuit together
Connections:
- net +5V: now also R401.2; no longer R401.1
- net ~RESET: now also R401.1; no longer R401.2
Changed lines of the file:
@@
 F 3 "~" H 2500 2300 50  0001 C CNN
 	1    2500 2300
-	1    0    0    -1
+	-1   0    0    1
 $EndComp
 $Comp
