File: Demultiplexer/InputSelect.kicad_sch (KiCad schematic)
At the start: 23 parts, among them SW201 SW_Push_Dual, SW202 SW_Push_Dual, U201 74HC14, U202 74HC74

Commit message: Working on routing
Connections:
- net GND: now also U201.13
- net ~{a_{0}}: now also R207.2; no longer R207.1
- net ~{a_{1}}: now also R208.2; no longer R208.1
- net at D203.2 (A): now also R207.1; no longer R207.2
- net at U202.11 (C): now also U201.6; no longer U201.12
- net at D204.2 (A): now also R208.1; no longer R208.2
- net at C204.1, R204.2: now also U201.5; no longer U201.13
Other:
- moved on the sheet: R207, R208, U201C, U201F
Changed lines of the file:
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@@
     (stroke (width 0) (type default) (color 0 0 0 0))
   )
-  (wire (pts (xy 17.78 152.4) (xy 19.05 152.4))
+  (wire (pts (xy 17.78 152.4) (xy 20.32 152.4))
     (stroke (width 0) (type default) (color 0 0 0 0))
   )
@@
     (pin "7")
   )
-  (symbol (lib_id "Device:R") (at 236.22 77.47 90) (unit 1)
+  (symbol (lib_id "Device:R") (at 236.22 77.47 270) (unit 1)
     (in_bom yes) (on_board yes) (fields_autoplaced)
     (property "Reference" "R207" (id 0) (at 236.22 71.12 90))
     (property "Value" "4k7" (id 1) (at 236.22 73.66 90))
-    (property "Footprint" "Resistor_THT:R_Axial_DIN0207_L6.3mm_D2.5mm_P7.62mm_Horizontal" (id 2) (at 236.22 79.248 90)
+    (property "Footprint" "Resistor_THT:R_Axial_DIN0207_L6.3mm_D2.5mm_P7.62mm_Horizontal" (id 2) (at 236.22 75.692 90)
       (effects (font (size 1.27 1.27)) hide)
     )
@@
     (pin "7")
   )
-  (symbol (lib_id "Device:R") (at 237.49 92.71 90) (unit 1)
+  (symbol (lib_id "Device:R") (at 237.49 92.71 270) (unit 1)
     (in_bom yes) (on_board yes) (fields_autoplaced)
     (property "Reference" "R208" (id 0) (at 237.49 86.36 90))
     (property "Value" "4k7" (id 1) (at 237.49 88.9 90))
-    (property "Footprint" "Resistor_THT:R_Axial_DIN0207_L6.3mm_D2.5mm_P7.62mm_Horizontal" (id 2) (at 237.49 94.488 90)
+    (property "Footprint" "Resistor_THT:R_Axial_DIN0207_L6.3mm_D2.5mm_P7.62mm_Horizontal" (id 2) (at 237.49 90.932 90)
       (effects (font (size 1.27 1.27)) hide)
     )
@@
     (pin "2")
   )
-  (symbol (lib_id "74xx:74HC14") (at 123.19 106.68 0) (unit 6)
-    (in_bom yes) (on_board yes) (fields_autoplaced)
-    (property "Reference" "U201" (id 0) (at 123.19 97.79 0))
-    (property "Value" "74HC14" (id 1) (at 123.19 100.33 0))
-    (property "Footprint" "" (id 2) (at 123.19 106.68 0)
-      (effects (font (size 1.27 1.27)) hide)
-    )
-    (property "Datasheet" "http://www.ti.com/lit/gpn/sn74HC14" (id 3) (at 123.19 106.68 0)
+  (symbol (lib_id "74xx:74HC14") (at 27.94 152.4 0) (unit 6)
+    (in_bom yes) (on_board yes) (fields_autoplaced)
+    (property "Reference" "U201" (id 0) (at 27.94 143.51 0))
+    (property "Value" "74HC14" (id 1) (at 27.94 146.05 0))
+    (property "Footprint" "" (id 2) (at 27.94 152.4 0)
+      (effects (font (size 1.27 1.27)) hide)
+    )
+    (property "Datasheet" "http://www.ti.com/lit/gpn/sn74HC14" (id 3) (at 27.94 152.4 0)
       (effects (font (size 1.27 1.27)) hide)
     )
@@
     (pin "1")
   )
-  (symbol (lib_id "74xx:74HC14") (at 27.94 152.4 0) (unit 3)
-    (in_bom yes) (on_board yes) (fields_autoplaced)
-    (property "Reference" "U201" (id 0) (at 27.94 143.51 0))
-    (property "Value" "74HC14" (id 1) (at 27.94 146.05 0))
-    (property "Footprint" "" (id 2) (at 27.94 152.4 0)
-      (effects (font (size 1.27 1.27)) hide)
-    )
-    (property "Datasheet" "http://www.ti.com/lit/gpn/sn74HC14" (id 3) (at 27.94 152.4 0)
-      (effects (font (size 1.27 1.27)) hide)
-    )
+  (symbol (lib_id "74xx:74HC14") (at 123.19 106.68 0) (unit 3)
+    (in_bom yes) (on_board yes) (fields_autoplaced)
+    (property "Reference" "U201" (id 0) (at 123.19 97.79 0))
+    (property "Value" "74HC14" (id 1) (at 123.19 100.33 0))
+    (property "Footprint" "" (id 2) (at 123.19 106.68 0)
+      (effects (font (size 1.27 1.27)) hide)
+    )
+    (property "Datasheet" "http://www.ti.com/lit/gpn/sn74HC14" (id 3) (at 123.19 106.68 0)
+      (effects (font (size 1.27 1.27)) hide)
+    )
