File: Demultiplexer/output.kicad_sch (KiCad schematic)
At the start: 8 parts, among them U401 74HC00, U402 74HC00

Commit message: Finish roughing out board
Parts:
- added C403, C404: 100nF, Capacitor_THT:C_Disc_D5.0mm_W2.5mm_P5.00mm, symbol Device:C
- added D403, D404: LED, LED_THT:LED_D5.0mm, symbol Device:LED
- added R403, R404: 4k7, Resistor_THT:R_Axial_DIN0207_L6.3mm_D2.5mm_P7.62mm_Horizontal, symbol Device:R
- added U403: 74HC00, symbol 74xx:74HC00
- added U404: 74HC00, Package_DIP:DIP-14_W7.62mm_Socket, symbol 74xx:74HC00
Connections:
- net +5V: now also C403.2, C404.2, U403.14 (VCC), U404.14 (VCC)
- net GND: now also C403.1, C404.1, D403.1 (K), D404.1 (K), U403.10, U403.12, U403.13, U403.7 (GND), U403.9, U404.10, U404.12, U404.13, U404.7 (GND), U404.9
- net INPUT: now also U403.1, U404.1
- new net: U403.3, U403.4, U403.5
- new net: D403.2 (A), R403.2
- new net: R404.1, U404.6
- new net: D404.2 (A), R404.2
- new net: U404.3, U404.4, U404.5
- new net: R403.1, U403.6
- new net SELECT2: U403.2
- new net SELECT3: U404.2
- no-connect marks 4 -> 8

Commit message: Working on routing
Connections:
- net INPUT: now also U401.2, U402.2, U403.2, U404.2; no longer U401.1, U402.1, U403.1, U404.1
- net SELECT0: now also U401.1; no longer U401.2
- net SELECT1: now also U402.1; no longer U402.2
- net SELECT2: now also U403.1; no longer U403.2
- net SELECT3: now also U404.1; no longer U404.2
Changed lines of the file:
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@@
   (junction (at 168.91 43.18) (diameter 0) (color 0 0 0 0)
   )
+  (junction (at 59.69 68.58) (diameter 0) (color 0 0 0 0)
+  )
+  (junction (at 59.69 90.17) (diameter 0) (color 0 0 0 0)
+  )
   (junction (at 170.18 134.62) (diameter 0) (color 0 0 0 0)
   )
@@
   (junction (at 97.79 87.63) (diameter 0) (color 0 0 0 0)
   )
-  (junction (at 58.42 40.64) (diameter 0) (color 0 0 0 0)
-  )
   (junction (at 168.91 78.74) (diameter 0) (color 0 0 0 0)
   )
-  (junction (at 58.42 63.5) (diameter 0) (color 0 0 0 0)
-  )
   (junction (at 168.91 25.4) (diameter 0) (color 0 0 0 0)
   )
@@
   (junction (at 207.01 99.06) (diameter 0) (color 0 0 0 0)
   )
+  (junction (at 59.69 45.72) (diameter 0) (color 0 0 0 0)
+  )
   (junction (at 168.91 38.1) (diameter 0) (color 0 0 0 0)
   )
@@
   )
   (junction (at 168.91 63.5) (diameter 0) (color 0 0 0 0)
-  )
-  (junction (at 58.42 85.09) (diameter 0) (color 0 0 0 0)
   )
   (no_connect (at 187.96 22.86))
@@
     (stroke (width 0) (type default) (color 0 0 0 0))
   )
-  (wire (pts (xy 58.42 63.5) (xy 74.93 63.5))
-    (stroke (width 0) (type default) (color 0 0 0 0))
-  )
   (wire (pts (xy 129.54 184.15) (xy 144.78 184.15))
     (stroke (width 0) (type default) (color 0 0 0 0))
@@
     (stroke (width 0) (type default) (color 0 0 0 0))
   )
-  (wire (pts (xy 58.42 63.5) (xy 58.42 85.09))
-    (stroke (width 0) (type default) (color 0 0 0 0))
-  )
   (wire (pts (xy 109.22 154.94) (xy 109.22 156.21))
     (stroke (width 0) (type default) (color 0 0 0 0))
@@
     (stroke (width 0) (type default) (color 0 0 0 0))
   )
+  (wire (pts (xy 59.69 90.17) (xy 74.93 90.17))
+    (stroke (width 0) (type default) (color 0 0 0 0))
+  )
   (wire (pts (xy 170.18 129.54) (xy 170.18 120.65))
     (stroke (width 0) (type default) (color 0 0 0 0))
@@
     (stroke (width 0) (type default) (color 0 0 0 0))
   )
+  (wire (pts (xy 59.69 45.72) (xy 59.69 68.58))
+    (stroke (width 0) (type default) (color 0 0 0 0))
+  )
   (wire (pts (xy 168.91 78.74) (xy 168.91 73.66))
     (stroke (width 0) (type default) (color 0 0 0 0))
@@
     (stroke (width 0) (type default) (color 0 0 0 0))
   )
-  (wire (pts (xy 54.61 45.72) (xy 74.93 45.72))
+  (wire (pts (xy 54.61 40.64) (xy 74.93 40.64))
     (stroke (width 0) (type default) (color 0 0 0 0))
   )
@@
     (stroke (width 0) (type default) (color 0 0 0 0))
   )
+  (wire (pts (xy 59.69 121.92) (xy 74.93 121.92))
+    (stroke (width 0) (type default) (color 0 0 0 0))
+  )
   (wire (pts (xy 168.91 58.42) (xy 172.72 58.42))
     (stroke (width 0) (type default) (color 0 0 0 0))
   )
+  (wire (pts (xy 59.69 68.58) (xy 74.93 68.58))
+    (stroke (width 0) (type default) (color 0 0 0 0))
+  )
   (wire (pts (xy 127 87.63) (xy 129.54 87.63))
     (stroke (width 0) (type default) (color 0 0 0 0))
@@
     (stroke (width 0) (type default) (color 0 0 0 0))
   )
-  (wire (pts (xy 58.42 85.09) (xy 74.93 85.09))
-    (stroke (width 0) (type default) (color 0 0 0 0))
-  )
   (wire (pts (xy 39.37 182.88) (xy 39.37 184.15))
     (stroke (width 0) (type default) (color 0 0 0 0))
@@
     (stroke (width 0) (type default) (color 0 0 0 0))
   )
+  (wire (pts (xy 59.69 45.72) (xy 74.93 45.72))
+    (stroke (width 0) (type default) (color 0 0 0 0))
+  )
+  (wire (pts (xy 59.69 68.58) (xy 59.69 90.17))
+    (stroke (width 0) (type default) (color 0 0 0 0))
+  )
   (wire (pts (xy 90.17 43.18) (xy 97.79 43.18))
     (stroke (width 0) (type default) (color 0 0 0 0))
@@
     (stroke (width 0) (type default) (color 0 0 0 0))
   )
-  (wire (pts (xy 58.42 40.64) (xy 58.42 63.5))
-    (stroke (width 0) (type default) (color 0 0 0 0))
-  )
   (wire (pts (xy 170.18 139.7) (xy 170.18 134.62))
     (stroke (width 0) (type default) (color 0 0 0 0))
@@
     (stroke (width 0) (type default) (color 0 0 0 0))
   )
-  (wire (pts (xy 54.61 40.64) (xy 58.42 40.64))
-    (stroke (width 0) (type default) (color 0 0 0 0))
-  )
   (wire (pts (xy 168.91 43.18) (xy 168.91 38.1))
     (stroke (width 0) (type default) (color 0 0 0 0))
@@
     (stroke (width 0) (type default) (color 0 0 0 0))
   )
-  (wire (pts (xy 54.61 90.17) (xy 74.93 90.17))
+  (wire (pts (xy 54.61 85.09) (xy 74.93 85.09))
     (stroke (width 0) (type default) (color 0 0 0 0))
   )
@@
     (stroke (width 0) (type default) (color 0 0 0 0))
   )
-  (wire (pts (xy 58.42 40.64) (xy 74.93 40.64))
+  (wire (pts (xy 54.61 45.72) (xy 59.69 45.72))
     (stroke (width 0) (type default) (color 0 0 0 0))
   )
@@
     (stroke (width 0) (type default) (color 0 0 0 0))
   )
+  (wire (pts (xy 59.69 90.17) (xy 59.69 121.92))
+    (stroke (width 0) (type default) (color 0 0 0 0))
+  )
   (wire (pts (xy 101.6 68.58) (xy 97.79 68.58))
     (stroke (width 0) (type default) (color 0 0 0 0))
@@
     (stroke (width 0) (type default) (color 0 0 0 0))
   )
-  (wire (pts (xy 58.42 116.84) (xy 74.93 116.84))
-    (stroke (width 0) (type default) (color 0 0 0 0))
-  )
-  (wire (pts (xy 53.34 121.92) (xy 74.93 121.92))
+  (wire (pts (xy 53.34 116.84) (xy 74.93 116.84))
     (stroke (width 0) (type default) (color 0 0 0 0))
   )
@@
     (stroke (width 0) (type default) (color 0 0 0 0))
   )
-  (wire (pts (xy 58.42 85.09) (xy 58.42 116.84))
-    (stroke (width 0) (type default) (color 0 0 0 0))
-  )
   (wire (pts (xy 93.98 176.53) (xy 93.98 184.15))
     (stroke (width 0) (type default) (color 0 0 0 0))
@@
     (stroke (width 0) (type default) (color 0 0 0 0))
   )
-  (wire (pts (xy 54.61 68.58) (xy 74.93 68.58))
+  (wire (pts (xy 54.61 63.5) (xy 74.93 63.5))
     (stroke (width 0) (type default) (color 0 0 0 0))
   )
@@
     (stroke (width 0) (type default) (color 0 0 0 0))
   )
-  (hierarchical_label "SELECT1" (shape input) (at 54.61 68.58 180)
-    (effects (font (size 1.27 1.27)) (justify right))
-  )
-  (hierarchical_label "SELECT2" (shape input) (at 54.61 90.17 180)
-    (effects (font (size 1.27 1.27)) (justify right))
-  )
-  (hierarchical_label "SELECT3" (shape input) (at 53.34 121.92 180)
-    (effects (font (size 1.27 1.27)) (justify right))
-  )
-  (hierarchical_label "INPUT" (shape input) (at 54.61 40.64 180)
-    (effects (font (size 1.27 1.27)) (justify right))
-  )
-  (hierarchical_label "SELECT0" (shape input) (at 54.61 45.72 180)
-    (effects (font (size 1.27 1.27)) (justify right))
-  )
+  (hierarchical_label "SELECT1" (shape input) (at 54.61 63.5 180)
+    (effects (font (size 1.27 1.27)) (justify right))
+  )
+  (hierarchical_label "SELECT2" (shape input) (at 54.61 85.09 180)
+    (effects (font (size 1.27 1.27)) (justify right))
+  )
+  (hierarchical_label "SELECT3" (shape input) (at 53.34 116.84 180)
+    (effects (font (size 1.27 1.27)) (justify right))
+  )
+  (hierarchical_label "INPUT" (shape input) (at 54.61 45.72 180)
+    (effects (font (size 1.27 1.27)) (justify right))
+  )
+  (hierarchical_label "SELECT0" (shape input) (at 54.61 40.64 180)
+    (effects (font (size 1.27 1.27)) (justify right))
+  )
