File: Johnson Counter/FlipflopUnit.kicad_sch (KiCad schematic)
At the start: 6 parts, among them U201 74HC74

Commit message: Getting flipflop board locations worked out
Parts:
- U201: footprint (none) -> Package_DIP:DIP-14_W7.62mm_Socket
Changed lines of the file:
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@@
       (effects (font (size 1.27 1.27)) (justify left))
     )
-    (property "Footprint" "" (id 2) (at 79.375 150.495 0)
+    (property "Footprint" "Package_DIP:DIP-14_W7.62mm_Socket" (id 2) (at 79.375 150.495 0)
       (effects (font (size 1.27 1.27)) hide)
     )
@@
       (effects (font (size 1.27 1.27)) (justify left))
     )
-    (property "Footprint" "" (id 2) (at 127 95.25 0)
+    (property "Footprint" "Package_DIP:DIP-14_W7.62mm_Socket" (id 2) (at 127 95.25 0)
       (effects (font (size 1.27 1.27)) hide)
     )
