File: Johnson Counter/clock.kicad_sch (KiCad schematic)
At the start: 6 parts

Commit message: Getting flipflop board locations worked out
Parts:
- gave numbers to parts that had none: 6
Changed lines of the file:
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@@
   (symbol (lib_id "Device:R") (at 48.895 58.42 0) (unit 1)
     (in_bom yes) (on_board yes)
-    (property "Reference" "R?" (id 0) (at 50.673 57.2516 0)
+    (property "Reference" "R601" (id 0) (at 50.673 57.2516 0)
       (effects (font (size 1.27 1.27)) (justify left))
     )
@@
   (symbol (lib_id "Device:C") (at 80.645 82.55 0) (unit 1)
     (in_bom yes) (on_board yes)
-    (property "Reference" "C?" (id 0) (at 77.724 83.7184 0)
+    (property "Reference" "C601" (id 0) (at 77.724 83.7184 0)
       (effects (font (size 1.27 1.27)) (justify right))
     )
@@
   (symbol (lib_id "power:+5V") (at 95.885 46.99 0) (unit 1)
     (in_bom yes) (on_board yes)
-    (property "Reference" "U?" (id 0) (at 95.885 50.8 0)
+    (property "Reference" "#U0102" (id 0) (at 95.885 50.8 0)
       (effects (font (size 1.27 1.27)) hide)
     )
@@
   (symbol (lib_id "power:GND") (at 95.885 93.98 0) (unit 1)
     (in_bom yes) (on_board yes)
-    (property "Reference" "U?" (id 0) (at 95.885 100.33 0)
+    (property "Reference" "#U0101" (id 0) (at 95.885 100.33 0)
       (effects (font (size 1.27 1.27)) hide)
     )
@@
   (symbol (lib_id "Switch:SW_Push") (at 48.895 76.2 270) (unit 1)
     (in_bom yes) (on_board yes)
-    (property "Reference" "U?" (id 0) (at 52.6542 75.0316 90)
+    (property "Reference" "SW601" (id 0) (at 52.6542 75.0316 90)
       (effects (font (size 1.27 1.27)) (justify left))
     )
@@
   (symbol (lib_id "Device:R") (at 120.015 59.69 0) (unit 1)
     (in_bom yes) (on_board yes)
-    (property "Reference" "R?" (id 0) (at 121.793 58.5216 0)
+    (property "Reference" "R602" (id 0) (at 121.793 58.5216 0)
       (effects (font (size 1.27 1.27)) (justify left))
     )
@@
   (symbol (lib_id "Timer:LM555xM") (at 95.885 71.12 0) (unit 1)
     (in_bom yes) (on_board yes)
-    (property "Reference" "U?" (id 0) (at 95.885 56.3626 0))
+    (property "Reference" "U601" (id 0) (at 95.885 56.3626 0))
     (property "Value" "LM555xM" (id 1) (at 95.885 58.674 0))
     (property "Footprint" "Package_DIP:DIP-8_W7.62mm_Socket" (id 2) (at 117.475 81.28 0)
@@
   (symbol (lib_id "power:+5V") (at 76.835 76.2 90) (unit 1)
     (in_bom yes) (on_board yes)
-    (property "Reference" "#PWR?" (id 0) (at 80.645 76.2 0)
+    (property "Reference" "#PWR0129" (id 0) (at 80.645 76.2 0)
       (effects (font (size 1.27 1.27)) hide)
     )
@@
   (symbol (lib_id "Device:C") (at 120.015 82.55 180) (unit 1)
     (in_bom yes) (on_board yes)
-    (property "Reference" "C?" (id 0) (at 117.094 83.7184 0)
+    (property "Reference" "C602" (id 0) (at 117.094 83.7184 0)
       (effects (font (size 1.27 1.27)) (justify left))
     )

Commit message: Finishing routing, silkscreen and mounting
Connections:
- net GND: now also C602.2; no longer C602.1
- net at R602.2, U601.6 (THR), U601.7 (DIS): now also C602.1; no longer C602.2
Other:
- moved on the sheet: C602
Changed lines of the file:
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@@
     (pin "1")
   )
-  (symbol (lib_id "Device:C") (at 120.015 82.55 180) (unit 1)
+  (symbol (lib_id "Device:C") (at 120.015 82.55 0) (unit 1)
     (in_bom yes) (on_board yes)
-    (property "Reference" "C602" (id 0) (at 117.094 83.7184 0)
+    (property "Reference" "C602" (id 0) (at 122.936 81.3816 0)
       (effects (font (size 1.27 1.27)) (justify left))
     )
-    (property "Value" "0.1u" (id 1) (at 117.094 81.407 0)
+    (property "Value" "0.1u" (id 1) (at 122.936 83.693 0)
       (effects (font (size 1.27 1.27)) (justify left))
     )
-    (property "Footprint" "Capacitor_THT:C_Disc_D4.7mm_W2.5mm_P5.00mm" (id 2) (at 119.0498 78.74 0)
+    (property "Footprint" "Capacitor_THT:C_Disc_D4.7mm_W2.5mm_P5.00mm" (id 2) (at 120.9802 86.36 0)
       (effects (font (size 1.27 1.27)) hide)
     )
