File: LFSR Disc 24/feedback.kicad_sch (KiCad schematic)
At the start: 3 parts, among them U501 74HC86, U502 74LS125

Commit message: More things assembling
Parts:
- added R501, R502: 100k, Resistor_THT:R_Axial_DIN0207_L6.3mm_D2.5mm_P7.62mm_Horizontal, symbol Device:R
- added SW201 (x2): SW_SPST, Button_Switch_THT:SW_PUSH_6mm, symbol Switch:SW_SPST
- R503: renamed from R501; value R -> 100k; footprint (none) -> Resistor_THT:R_Axial_DIN0207_L6.3mm_D2.5mm_P7.62mm_Horizontal
- U502: value 74LS125 -> 74HCT125
Connections:
- net +5V: now also U502.9, SW201.1 (A), SW201.1 (A)
- net GND: now also R503.2, R501.2, R502.2
- net at R503.1: now also U502.5, SW201.2 (B)
- net ~{FEEDBACK}: now reaches U502.10
- net ~{FEEDBACK}: now also R501.1, SW201.2 (B)
- net ~{MANUAL}: now reaches U502.8
- net ~{MANUAL}: now also R502.1
Other:
- moved on the sheet: U502C

Commit message: Board layout and schematic tweaks
Connections:
- net IN0: now also U501.5; no longer U501.1
- net IN1: now also U501.4; no longer U501.2
- net IN2: now also U501.2; no longer U501.4
- net IN3: now also U501.1; no longer U501.5
- net NXTBIT: now also U502.11; no longer U502.6
- net ~{FEEDBACK}: now also U502.1
- net ~{MANUAL}: now also U502.13
- net at R503.1, SW201.2 (B): now also U502.12; no longer U502.5
- net at U501.6: now also U501.9; no longer U501.10
- net at U501.3: now also U501.10; no longer U501.9
Other:
- moved on the sheet: U501A, U501B, U502B, U502D

Commit message: Final routing
Connections:
- net GND: now also U501.12, U501.13, U502.4, U502.5
- no-connect marks 0 -> 2
Changed lines of the file:
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@@
   (junction (at 118.11 93.98) (diameter 0) (color 0 0 0 0)
   )
+  (junction (at 158.75 167.64) (diameter 0) (color 0 0 0 0)
+  )
   (junction (at 77.47 110.49) (diameter 0) (color 0 0 0 0)
   )
@@
   (junction (at 77.47 93.98) (diameter 0) (color 0 0 0 0)
   )
+  (junction (at 100.33 171.45) (diameter 0) (color 0 0 0 0)
+  )
+  (no_connect (at 120.65 168.91))
+  (no_connect (at 177.8 160.02))
   (wire (pts (xy 255.27 91.44) (xy 246.38 91.44))
     (stroke (width 0) (type default))
@@
     (stroke (width 0) (type default))
   )
+  (wire (pts (xy 170.18 166.37) (xy 170.18 167.64))
+    (stroke (width 0) (type default))
+  )
+  (wire (pts (xy 100.33 166.37) (xy 105.41 166.37))
+    (stroke (width 0) (type default))
+  )
   (wire (pts (xy 209.55 74.93) (xy 209.55 78.74))
     (stroke (width 0) (type default))
   )
+  (wire (pts (xy 158.75 160.02) (xy 162.56 160.02))
+    (stroke (width 0) (type default))
+  )
   (wire (pts (xy 255.27 66.04) (xy 266.7 66.04))
     (stroke (width 0) (type default))
@@
     (stroke (width 0) (type default))
   )
+  (wire (pts (xy 158.75 167.64) (xy 158.75 160.02))
+    (stroke (width 0) (type default))
+  )
   (wire (pts (xy 128.27 83.82) (xy 133.35 83.82))
     (stroke (width 0) (type default))
@@
     (stroke (width 0) (type default))
   )
+  (wire (pts (xy 100.33 171.45) (xy 105.41 171.45))
+    (stroke (width 0) (type default))
+  )
   (wire (pts (xy 177.8 53.34) (xy 182.88 53.34))
     (stroke (width 0) (type default))
@@
     (stroke (width 0) (type default))
   )
+  (wire (pts (xy 158.75 170.18) (xy 158.75 167.64))
+    (stroke (width 0) (type default))
+  )
   (wire (pts (xy 107.95 110.49) (xy 123.19 110.49))
     (stroke (width 0) (type default))
@@
   )
   (wire (pts (xy 77.47 93.98) (xy 77.47 97.79))
+    (stroke (width 0) (type default))
+  )
+  (wire (pts (xy 100.33 171.45) (xy 100.33 166.37))
+    (stroke (width 0) (type default))
+  )
+  (wire (pts (xy 100.33 177.8) (xy 100.33 171.45))
+    (stroke (width 0) (type default))
+  )
+  (wire (pts (xy 158.75 167.64) (xy 170.18 167.64))
     (stroke (width 0) (type default))
   )
@@
     )
   )
+  (symbol (lib_id "power:GND") (at 158.75 170.18 0) (unit 1)
+    (in_bom yes) (on_board yes) (dnp no) (fields_autoplaced)
+    (property "Reference" "#PWR0509" (at 158.75 176.53 0)
+      (effects (font (size 1.27 1.27)) hide)
+    )
+    (property "Value" "GND" (at 158.75 175.26 0)
+      (effects (font (size 1.27 1.27)))
+    )
+    (property "Footprint" "" (at 158.75 170.18 0)
+      (effects (font (size 1.27 1.27)) hide)
+    )
+    (property "Datasheet" "" (at 158.75 170.18 0)
+      (effects (font (size 1.27 1.27)) hide)
+    )
+    (pin "1")
+    (instances
+      (project "LFSR Disc 24"
+        (path "/d11adbca-5bbf-4b99-b4dc-9e7e9b691814/36102b2f-4921-453b-a894-0645b75cde18/76cd073a-97c1-4f51-b028-2b34aeb12b55"
+          (reference "#PWR0509") (unit 1)
+        )
+      )
+    )
+  )
   (symbol (lib_id "power:GND") (at 133.35 83.82 90) (unit 1)
     (in_bom yes) (on_board yes) (dnp no) (fields_autoplaced)
@@
         )
       )
+    )
+  )
+  (symbol (lib_id "power:GND") (at 100.33 177.8 0) (unit 1)
+    (in_bom yes) (on_board yes) (dnp no) (fields_autoplaced)
+    (property "Reference" "#PWR0508" (at 100.33 184.15 0)
+      (effects (font (size 1.27 1.27)) hide)
+    )
+    (property "Value" "GND" (at 100.33 182.88 0)
+      (effects (font (size 1.27 1.27)))
+    )
+    (property "Footprint" "" (at 100.33 177.8 0)
+      (effects (font (size 1.27 1.27)) hide)
+    )
+    (property "Datasheet" "" (at 100.33 177.8 0)
+      (effects (font (size 1.27 1.27)) hide)
+    )
+    (pin "1")
+    (instances
+      (project "LFSR Disc 24"
+        (path "/d11adbca-5bbf-4b99-b4dc-9e7e9b691814/36102b2f-4921-453b-a894-0645b75cde18/76cd073a-97c1-4f51-b028-2b34aeb12b55"
+          (reference "#PWR0508") (unit 1)
+        )
+      )
