File: LFSR Disc 24/leds.kicad_sch (KiCad schematic)
At the start: 48 parts

Commit message: Filling things out a little
Parts:
- R301, R302, R303, R304, R305, R306, R307, R308, R309, R310, R311, R312, R313, R314, R315, R316, R317, R318, R319, R320, R321, R322, R323, R324: value R -> 4k7
Changed lines of the file:
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@@
     (stroke (width 0) (type default))
   )
-  (label "LED3" (at 46.99 48.26 0)
+  (label "LED3" (at 46.99 48.26 0) (fields_autoplaced)
     (effects (font (size 1.27 1.27)) (justify left bottom))
   )
-  (label "LED4" (at 46.99 59.69 0)
+  (label "LED4" (at 46.99 59.69 0) (fields_autoplaced)
     (effects (font (size 1.27 1.27)) (justify left bottom))
   )
-  (label "LED7" (at 46.99 95.25 0)
+  (label "LED7" (at 46.99 95.25 0) (fields_autoplaced)
     (effects (font (size 1.27 1.27)) (justify left bottom))
   )
-  (label "LED2" (at 46.99 36.83 0)
+  (label "LED2" (at 46.99 36.83 0) (fields_autoplaced)
     (effects (font (size 1.27 1.27)) (justify left bottom))
   )
-  (label "LED5" (at 46.99 72.39 0)
+  (label "LED5" (at 46.99 72.39 0) (fields_autoplaced)
     (effects (font (size 1.27 1.27)) (justify left bottom))
   )
-  (label "LED6" (at 46.99 83.82 0)
+  (label "LED6" (at 46.99 83.82 0) (fields_autoplaced)
     (effects (font (size 1.27 1.27)) (justify left bottom))
   )
-  (label "LED8" (at 46.99 106.68 0)
+  (label "LED8" (at 46.99 106.68 0) (fields_autoplaced)
     (effects (font (size 1.27 1.27)) (justify left bottom))
   )
-  (label "LED1" (at 46.99 25.4 0)
+  (label "LED1" (at 46.99 25.4 0) (fields_autoplaced)
     (effects (font (size 1.27 1.27)) (justify left bottom))
   )
-  (label "LED16" (at 153.67 59.69 0)
+  (label "LED16" (at 153.67 59.69 0) (fields_autoplaced)
     (effects (font (size 1.27 1.27)) (justify left bottom))
   )
@@
       (effects (font (size 1.27 1.27)))
     )
-    (property "Value" "R" (at 85.09 125.73 90)
+    (property "Value" "4k7" (at 85.09 125.73 90)
       (effects (font (size 1.27 1.27)))
     )
@@
       (effects (font (size 1.27 1.27)))
     )
-    (property "Value" "R" (at 186.69 91.44 90)
+    (property "Value" "4k7" (at 186.69 91.44 90)
       (effects (font (size 1.27 1.27)))
     )
@@
       (effects (font (size 1.27 1.27)))
     )
-    (property "Value" "R" (at 85.09 102.87 90)
+    (property "Value" "4k7" (at 85.09 102.87 90)
       (effects (font (size 1.27 1.27)))
     )
@@
       (effects (font (size 1.27 1.27)))
     )
-    (property "Value" "R" (at 85.09 137.16 90)
+    (property "Value" "4k7" (at 85.09 137.16 90)
       (effects (font (size 1.27 1.27)))
     )
@@
       (effects (font (size 1.27 1.27)))
     )
-    (property "Value" "R" (at 186.69 80.01 90)
+    (property "Value" "4k7" (at 186.69 80.01 90)
       (effects (font (size 1.27 1.27)))
     )
@@
       (effects (font (size 1.27 1.27)))
     )
-    (property "Value" "R" (at 85.09 114.3 90)
+    (property "Value" "4k7" (at 85.09 114.3 90)
       (effects (font (size 1.27 1.27)))
     )
@@
       (effects (font (size 1.27 1.27)))
     )
-    (property "Value" "R" (at 186.69 55.88 90)
+    (property "Value" "4k7" (at 186.69 55.88 90)
       (effects (font (size 1.27 1.27)))
     )
@@
       (effects (font (size 1.27 1.27)))
     )
-    (property "Value" "R" (at 85.09 44.45 90)
+    (property "Value" "4k7" (at 85.09 44.45 90)
       (effects (font (size 1.27 1.27)))
     )
@@
       (effects (font (size 1.27 1.27)))
     )
-    (property "Value" "R" (at 85.09 91.44 90)
+    (property "Value" "4k7" (at 85.09 91.44 90)
       (effects (font (size 1.27 1.27)))
     )
@@
       (effects (font (size 1.27 1.27)))
     )
-    (property "Value" "R" (at 85.09 80.01 90)
+    (property "Value" "4k7" (at 85.09 80.01 90)
       (effects (font (size 1.27 1.27)))
     )
@@
       (effects (font (size 1.27 1.27)))
     )
-    (property "Value" "R" (at 186.69 125.73 90)
+    (property "Value" "4k7" (at 186.69 125.73 90)
       (effects (font (size 1.27 1.27)))
     )
@@
       (effects (font (size 1.27 1.27)))
     )
-    (property "Value" "R" (at 186.69 137.16 90)
+    (property "Value" "4k7" (at 186.69 137.16 90)
       (effects (font (size 1.27 1.27)))
     )
@@
       (effects (font (size 1.27 1.27)))
     )
-    (property "Value" "R" (at 186.69 68.58 90)
+    (property "Value" "4k7" (at 186.69 68.58 90)
       (effects (font (size 1.27 1.27)))
     )
@@
       (effects (font (size 1.27 1.27)))
     )
-    (property "Value" "R" (at 186.69 102.87 90)
+    (property "Value" "4k7" (at 186.69 102.87 90)
       (effects (font (size 1.27 1.27)))
     )
@@
       (effects (font (size 1.27 1.27)))
     )
-    (property "Value" "R" (at 85.09 68.58 90)
+    (property "Value" "4k7" (at 85.09 68.58 90)
       (effects (font (size 1.27 1.27)))
     )
@@
       (effects (font (size 1.27 1.27)))
     )
-    (property "Value" "R" (at 186.69 21.59 90)
+    (property "Value" "4k7" (at 186.69 21.59 90)
       (effects (font (size 1.27 1.27)))
     )
@@
       (effects (font (size 1.27 1.27)))
     )
-    (property "Value" "R" (at 186.69 33.02 90)
+    (property "Value" "4k7" (at 186.69 33.02 90)
       (effects (font (size 1.27 1.27)))
     )
@@
       (effects (font (size 1.27 1.27)))
     )
-    (property "Value" "R" (at 186.69 148.59 90)
+    (property "Value" "4k7" (at 186.69 148.59 90)
       (effects (font (size 1.27 1.27)))
     )
@@
       (effects (font (size 1.27 1.27)))
     )
-    (property "Value" "R" (at 186.69 44.45 90)
+    (property "Value" "4k7" (at 186.69 44.45 90)
       (effects (font (size 1.27 1.27)))
     )
@@
       (effects (font (size 1.27 1.27)))
     )
-    (property "Value" "R" (at 85.09 33.02 90)
+    (property "Value" "4k7" (at 85.09 33.02 90)
       (effects (font (size 1.27 1.27)))
     )
@@
       (effects (font (size 1.27 1.27)))
     )
-    (property "Value" "R" (at 186.69 114.3 90)
+    (property "Value" "4k7" (at 186.69 114.3 90)
       (effects (font (size 1.27 1.27)))
     )
@@
       (effects (font (size 1.27 1.27)))
     )
-    (property "Value" "R" (at 85.09 148.59 90)
+    (property "Value" "4k7" (at 85.09 148.59 90)
       (effects (font (size 1.27 1.27)))
     )
@@
       (effects (font (size 1.27 1.27)))
     )
-    (property "Value" "R" (at 85.09 55.88 90)
+    (property "Value" "4k7" (at 85.09 55.88 90)
       (effects (font (size 1.27 1.27)))
     )
@@
       (effects (font (size 1.27 1.27)))
     )
-    (property "Value" "R" (at 85.09 21.59 90)
-      (effects (font (size 1.27 1.27)))
-    )
+    (property "Value" "4k7" (at 85.09 21.59 90)
+      (effects (font (size 1.27 1.27)))
+    )

Commit message: More things assembling
Connections:
- net LED10: now reaches D310.2 (A)
- net LED15: now reaches D315.2 (A)
- net LED12: now reaches D312.2 (A)
- net LED9: now reaches D309.2 (A)
- net LED11: now reaches D311.2 (A)
- net LED14: now reaches D314.2 (A)
- net LED13: now reaches D313.2 (A)
Changed lines of the file:
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@@
+    (stroke (width 0) (type default))
+  )
+  (bus_entry (at 44.45 120.65) (size 2.54 -2.54)
+    (stroke (width 0) (type default))
+  )
+  (bus_entry (at 44.45 143.51) (size 2.54 -2.54)
+    (stroke (width 0) (type default))
+  )
+  (bus_entry (at 44.45 132.08) (size 2.54 -2.54)
     (stroke (width 0) (type default))
   )
@@
     (stroke (width 0) (type default))
   )
+  (bus_entry (at 151.13 27.94) (size 2.54 -2.54)
+    (stroke (width 0) (type default))
+  )
+  (bus_entry (at 151.13 50.8) (size 2.54 -2.54)
+    (stroke (width 0) (type default))
+  )
   (bus_entry (at 44.45 39.37) (size 2.54 -2.54)
     (stroke (width 0) (type default))
@@
     (stroke (width 0) (type default))
   )
+  (bus_entry (at 44.45 154.94) (size 2.54 -2.54)
+    (stroke (width 0) (type default))
+  )
+  (bus_entry (at 151.13 39.37) (size 2.54 -2.54)
+    (stroke (width 0) (type default))
+  )
   (bus_entry (at 151.13 62.23) (size 2.54 -2.54)
     (stroke (width 0) (type default))
   )
+  (wire (pts (xy 46.99 118.11) (xy 64.77 118.11))
+    (stroke (width 0) (type default))
+  )
   (wire (pts (xy 88.9 95.25) (xy 95.25 95.25))
     (stroke (width 0) (type default))
   )
+  (bus (pts (xy 151.13 39.37) (xy 151.13 50.8))
+    (stroke (width 0) (type default))
+  )
   (wire (pts (xy 95.25 25.4) (xy 95.25 36.83))
     (stroke (width 0) (type default))
@@
     (stroke (width 0) (type default))
   )
+  (wire (pts (xy 153.67 36.83) (xy 166.37 36.83))
+    (stroke (width 0) (type default))
+  )
   (wire (pts (xy 88.9 72.39) (xy 95.25 72.39))
     (stroke (width 0) (type default))
@@
     (stroke (width 0) (type default))
   )
-  (bus (pts (xy 151.13 25.4) (xy 151.13 62.23))
-    (stroke (width 0) (type default))
-  )
   (wire (pts (xy 173.99 36.83) (xy 182.88 36.83))
     (stroke (width 0) (type default))
@@
     (stroke (width 0) (type default))
   )
-  (bus (pts (xy 44.45 109.22) (xy 44.45 179.07))
+  (bus (pts (xy 44.45 109.22) (xy 44.45 120.65))
     (stroke (width 0) (type default))
   )
@@
     (stroke (width 0) (type default))
   )
+  (wire (pts (xy 46.99 152.4) (xy 64.77 152.4))
+    (stroke (width 0) (type default))
+  )
   (bus (pts (xy 44.45 39.37) (xy 44.45 50.8))
     (stroke (width 0) (type default))
@@
     (stroke (width 0) (type default))
   )
+  (wire (pts (xy 46.99 140.97) (xy 64.77 140.97))
+    (stroke (width 0) (type default))
+  )
   (wire (pts (xy 196.85 95.25) (xy 196.85 106.68))
     (stroke (width 0) (type default))
@@
     (stroke (width 0) (type default))
   )
+  (bus (pts (xy 44.45 120.65) (xy 44.45 132.08))
+    (stroke (width 0) (type default))
+  )
   (wire (pts (xy 173.99 106.68) (xy 182.88 106.68))
     (stroke (width 0) (type default))
@@
     (stroke (width 0) (type default))
   )
+  (bus (pts (xy 44.45 154.94) (xy 44.45 179.07))
+    (stroke (width 0) (type default))
+  )
   (bus (pts (xy 44.45 74.93) (xy 44.45 86.36))
     (stroke (width 0) (type default))
@@
     (stroke (width 0) (type default))
   )
+  (wire (pts (xy 46.99 129.54) (xy 64.77 129.54))
+    (stroke (width 0) (type default))
+  )
+  (bus (pts (xy 151.13 50.8) (xy 151.13 62.23))
+    (stroke (width 0) (type default))
+  )
+  (bus (pts (xy 151.13 27.94) (xy 151.13 39.37))
+    (stroke (width 0) (type default))
+  )
   (wire (pts (xy 46.99 59.69) (xy 64.77 59.69))
     (stroke (width 0) (type default))
   )
+  (bus (pts (xy 44.45 143.51) (xy 44.45 154.94))
+    (stroke (width 0) (type default))
+  )
   (bus (pts (xy 44.45 50.8) (xy 44.45 62.23))
     (stroke (width 0) (type default))
@@
     (stroke (width 0) (type default))
   )
+  (wire (pts (xy 153.67 25.4) (xy 166.37 25.4))
+    (stroke (width 0) (type default))
+  )
   (bus (pts (xy 44.45 86.36) (xy 44.45 97.79))
     (stroke (width 0) (type default))
@@
     (stroke (width 0) (type default))
   )
+  (bus (pts (xy 44.45 132.08) (xy 44.45 143.51))
+    (stroke (width 0) (type default))
+  )
   (wire (pts (xy 46.99 25.4) (xy 64.77 25.4))
     (stroke (width 0) (type default))
@@
     (stroke (width 0) (type default))
   )
+  (wire (pts (xy 153.67 48.26) (xy 166.37 48.26))
+    (stroke (width 0) (type default))
+  )
   (wire (pts (xy 190.5 106.68) (xy 196.85 106.68))
     (stroke (width 0) (type default))
@@
     (effects (font (size 1.27 1.27)) (justify left bottom))
   )
+  (label "LED13" (at 153.67 25.4 0)
+    (effects (font (size 1.27 1.27)) (justify left bottom))
+  )
+  (label "LED14" (at 153.67 36.83 0)
+    (effects (font (size 1.27 1.27)) (justify left bottom))
+  )
+  (label "LED11" (at 46.99 140.97 0)
+    (effects (font (size 1.27 1.27)) (justify left bottom))
+  )
   (label "LED7" (at 46.99 95.25 0) (fields_autoplaced)
     (effects (font (size 1.27 1.27)) (justify left bottom))
@@
     (effects (font (size 1.27 1.27)) (justify left bottom))
   )
+  (label "LED10" (at 46.99 129.54 0)
+    (effects (font (size 1.27 1.27)) (justify left bottom))
+  )
+  (label "LED12" (at 46.99 152.4 0)
+    (effects (font (size 1.27 1.27)) (justify left bottom))
+  )
+  (label "LED15" (at 153.67 48.26 0)
+    (effects (font (size 1.27 1.27)) (justify left bottom))
+  )
+  (label "LED9" (at 46.99 118.11 0)
+    (effects (font (size 1.27 1.27)) (justify left bottom))
+  )

Commit message: Board layout and schematic tweaks
Connections:
- net LED22: now reaches D322.2 (A)
- net LED19: now reaches D319.2 (A)
- net LED23: now reaches D323.2 (A)
- net LED20: now reaches D320.2 (A)
- net LED24: now reaches D324.2 (A)
- net LED17: now reaches D317.2 (A)
- net LED21: now reaches D321.2 (A)
- net LED18: now reaches D318.2 (A)
Changed lines of the file:
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@@
+    (stroke (width 0) (type default))
+  )
+  (bus_entry (at 151.13 74.93) (size 2.54 -2.54)
     (stroke (width 0) (type default))
   )
@@
     (stroke (width 0) (type default))
   )
+  (bus_entry (at 151.13 97.79) (size 2.54 -2.54)
+    (stroke (width 0) (type default))
+  )
   (bus_entry (at 44.45 27.94) (size 2.54 -2.54)
     (stroke (width 0) (type default))
@@
     (stroke (width 0) (type default))
   )
+  (bus_entry (at 151.13 120.65) (size 2.54 -2.54)
+    (stroke (width 0) (type default))
+  )
   (bus_entry (at 151.13 39.37) (size 2.54 -2.54)
     (stroke (width 0) (type default))
   )
+  (bus_entry (at 151.13 143.51) (size 2.54 -2.54)
+    (stroke (width 0) (type default))
+  )
+  (bus_entry (at 151.13 109.22) (size 2.54 -2.54)
+    (stroke (width 0) (type default))
+  )
+  (bus_entry (at 151.13 132.08) (size 2.54 -2.54)
+    (stroke (width 0) (type default))
+  )
+  (bus_entry (at 151.13 86.36) (size 2.54 -2.54)
+    (stroke (width 0) (type default))
+  )
   (bus_entry (at 151.13 62.23) (size 2.54 -2.54)
     (stroke (width 0) (type default))
   )
+  (bus_entry (at 151.13 154.94) (size 2.54 -2.54)
+    (stroke (width 0) (type default))
+  )
   (wire (pts (xy 46.99 118.11) (xy 64.77 118.11))
     (stroke (width 0) (type default))
@@
     (stroke (width 0) (type default))
   )
+  (wire (pts (xy 153.67 118.11) (xy 166.37 118.11))
+    (stroke (width 0) (type default))
+  )
   (wire (pts (xy 190.5 129.54) (xy 196.85 129.54))
     (stroke (width 0) (type default))
@@
     (stroke (width 0) (type default))
   )
+  (bus (pts (xy 151.13 154.94) (xy 151.13 179.07))
+    (stroke (width 0) (type default))
+  )
+  (wire (pts (xy 153.67 72.39) (xy 166.37 72.39))
+    (stroke (width 0) (type default))
+  )
   (wire (pts (xy 153.67 36.83) (xy 166.37 36.83))
     (stroke (width 0) (type default))
@@
     (stroke (width 0) (type default))
   )
+  (wire (pts (xy 153.67 83.82) (xy 166.37 83.82))
+    (stroke (width 0) (type default))
+  )
   (wire (pts (xy 88.9 48.26) (xy 95.25 48.26))
     (stroke (width 0) (type default))
@@
     (stroke (width 0) (type default))
   )
+  (bus (pts (xy 151.13 109.22) (xy 151.13 120.65))
+    (stroke (width 0) (type default))
+  )
   (wire (pts (xy 190.5 118.11) (xy 196.85 118.11))
     (stroke (width 0) (type default))
@@
     (stroke (width 0) (type default))
   )
+  (wire (pts (xy 153.67 129.54) (xy 166.37 129.54))
+    (stroke (width 0) (type default))
+  )
   (wire (pts (xy 196.85 95.25) (xy 196.85 106.68))
     (stroke (width 0) (type default))
@@
     (stroke (width 0) (type default))
   )
-  (bus (pts (xy 151.13 62.23) (xy 151.13 179.07))
+  (bus (pts (xy 151.13 62.23) (xy 151.13 74.93))
     (stroke (width 0) (type default))
   )
@@
     (stroke (width 0) (type default))
   )
+  (bus (pts (xy 151.13 132.08) (xy 151.13 143.51))
+    (stroke (width 0) (type default))
+  )
   (wire (pts (xy 95.25 59.69) (xy 95.25 72.39))
     (stroke (width 0) (type default))
@@
     (stroke (width 0) (type default))
   )
+  (wire (pts (xy 153.67 95.25) (xy 166.37 95.25))
+    (stroke (width 0) (type default))
+  )
   (wire (pts (xy 46.99 95.25) (xy 64.77 95.25))
     (stroke (width 0) (type default))
@@
     (stroke (width 0) (type default))
   )
+  (bus (pts (xy 151.13 143.51) (xy 151.13 154.94))
+    (stroke (width 0) (type default))
+  )
   (wire (pts (xy 196.85 36.83) (xy 196.85 48.26))
     (stroke (width 0) (type default))
@@
     (stroke (width 0) (type default))
   )
+  (wire (pts (xy 153.67 152.4) (xy 166.37 152.4))
+    (stroke (width 0) (type default))
+  )
   (wire (pts (xy 72.39 152.4) (xy 81.28 152.4))
     (stroke (width 0) (type default))
   )
+  (bus (pts (xy 151.13 97.79) (xy 151.13 109.22))
+    (stroke (width 0) (type default))
+  )
   (wire (pts (xy 190.5 25.4) (xy 196.85 25.4))
     (stroke (width 0) (type default))
@@
     (stroke (width 0) (type default))
   )
+  (bus (pts (xy 151.13 74.93) (xy 151.13 86.36))
+    (stroke (width 0) (type default))
+  )
   (bus (pts (xy 151.13 27.94) (xy 151.13 39.37))
     (stroke (width 0) (type default))
@@
     (stroke (width 0) (type default))
   )
+  (bus (pts (xy 151.13 86.36) (xy 151.13 97.79))
+    (stroke (width 0) (type default))
+  )
   (wire (pts (xy 72.39 140.97) (xy 81.28 140.97))
     (stroke (width 0) (type default))
@@
     (stroke (width 0) (type default))
   )
+  (wire (pts (xy 153.67 106.68) (xy 166.37 106.68))
+    (stroke (width 0) (type default))
+  )
   (wire (pts (xy 153.67 25.4) (xy 166.37 25.4))
     (stroke (width 0) (type default))
@@
     (stroke (width 0) (type default))
   )
+  (bus (pts (xy 151.13 120.65) (xy 151.13 132.08))
+    (stroke (width 0) (type default))
+  )
   (wire (pts (xy 196.85 129.54) (xy 196.85 140.97))
     (stroke (width 0) (type default))
@@
     (stroke (width 0) (type default))
   )
+  (wire (pts (xy 153.67 140.97) (xy 166.37 140.97))
+    (stroke (width 0) (type default))
+  )
   (wire (pts (xy 190.5 152.4) (xy 196.85 152.4))
     (stroke (width 0) (type default))
@@
     (effects (font (size 1.27 1.27)) (justify left bottom))
   )
-  (label "LED13" (at 153.67 25.4 0)
-    (effects (font (size 1.27 1.27)) (justify left bottom))
-  )
-  (label "LED14" (at 153.67 36.83 0)
-    (effects (font (size 1.27 1.27)) (justify left bottom))
-  )
-  (label "LED11" (at 46.99 140.97 0)
+  (label "LED13" (at 153.67 25.4 0) (fields_autoplaced)
+    (effects (font (size 1.27 1.27)) (justify left bottom))
+  )
+  (label "LED14" (at 153.67 36.83 0) (fields_autoplaced)
+    (effects (font (size 1.27 1.27)) (justify left bottom))
+  )
+  (label "LED22" (at 153.67 129.54 0)
+    (effects (font (size 1.27 1.27)) (justify left bottom))
+  )
+  (label "LED11" (at 46.99 140.97 0) (fields_autoplaced)
+    (effects (font (size 1.27 1.27)) (justify left bottom))
+  )
+  (label "LED19" (at 153.67 95.25 0)
     (effects (font (size 1.27 1.27)) (justify left bottom))
   )
@@
     (effects (font (size 1.27 1.27)) (justify left bottom))
   )
+  (label "LED18" (at 153.67 83.82 0)
+    (effects (font (size 1.27 1.27)) (justify left bottom))
+  )
+  (label "LED21" (at 153.67 118.11 0)
+    (effects (font (size 1.27 1.27)) (justify left bottom))
+  )
   (label "LED6" (at 46.99 83.82 0) (fields_autoplaced)
     (effects (font (size 1.27 1.27)) (justify left bottom))
@@
     (effects (font (size 1.27 1.27)) (justify left bottom))
   )
+  (label "LED17" (at 153.67 72.39 0)
+    (effects (font (size 1.27 1.27)) (justify left bottom))
+  )
   (label "LED1" (at 46.99 25.4 0) (fields_autoplaced)
     (effects (font (size 1.27 1.27)) (justify left bottom))
   )
-  (label "LED10" (at 46.99 129.54 0)
-    (effects (font (size 1.27 1.27)) (justify left bottom))
-  )
-  (label "LED12" (at 46.99 152.4 0)
-    (effects (font (size 1.27 1.27)) (justify left bottom))
-  )
-  (label "LED15" (at 153.67 48.26 0)
-    (effects (font (size 1.27 1.27)) (justify left bottom))
-  )
-  (label "LED9" (at 46.99 118.11 0)
+  (label "LED10" (at 46.99 129.54 0) (fields_autoplaced)
+    (effects (font (size 1.27 1.27)) (justify left bottom))
+  )
+  (label "LED12" (at 46.99 152.4 0) (fields_autoplaced)
+    (effects (font (size 1.27 1.27)) (justify left bottom))
+  )
+  (label "LED20" (at 153.67 106.68 0)
+    (effects (font (size 1.27 1.27)) (justify left bottom))
+  )
+  (label "LED24" (at 153.67 152.4 0)
+    (effects (font (size 1.27 1.27)) (justify left bottom))
+  )
+  (label "LED15" (at 153.67 48.26 0) (fields_autoplaced)
+    (effects (font (size 1.27 1.27)) (justify left bottom))
+  )
+  (label "LED9" (at 46.99 118.11 0) (fields_autoplaced)
     (effects (font (size 1.27 1.27)) (justify left bottom))
   )
@@
     (effects (font (size 1.27 1.27)) (justify left bottom))
   )
+  (label "LED23" (at 153.67 140.97 0)
+    (effects (font (size 1.27 1.27)) (justify left bottom))
+  )
