File: LFSR Disc 24/shiftregisters.kicad_sch (KiCad schematic)
At the start: 3 parts, among them U201 74HC164, U202 74HC164, U203 74HC164

Commit message: Filling things out a little
Connections:
- net CLK: now reaches U201.8 (CP)
- net CLK: now also U202.8 (CP), U203.8 (CP)
- net LED21: now reaches U203.10 (Q4)
- net LED22: now reaches U203.11 (Q5)
- net LED23: now reaches U203.12 (Q6)
- net LED24: now reaches U203.13 (Q7)
- net LED17: now reaches U203.3 (Q0)
- net LED18: now reaches U203.4 (Q1)
- net LED19: now reaches U203.5 (Q2)
- net LED20: now reaches U203.6 (Q3)
Other:
- added sheet Feedback (feedback.kicad_sch)

Commit message: More things assembling
Parts:
- added C802 (x3): 0.1u, Capacitor_THT:C_Disc_D4.3mm_W1.9mm_P5.00mm, symbol Device:C
Connections:
- net +5V: now also C802.2, C802.2, C802.2
- net GND: now also C802.1, C802.1, C802.1
- net Feedback/NXTBIT: now reaches U201.1 (DSA)
- net Feedback/NXTBIT: now also U201.2 (DSB)
Other:
- sheet Feedback ports: added IN0, IN1, IN2, IN3, NXTBIT; removed none

Commit message: Board layout and schematic tweaks
Changed lines of the file:
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@@
+    (stroke (width 0) (type default))
+  )
+  (wire (pts (xy 20.32 38.1) (xy 26.67 38.1))
     (stroke (width 0) (type default))
   )
@@
     (stroke (width 0) (type default))
   )
+  (wire (pts (xy 20.32 35.56) (xy 26.67 35.56))
+    (stroke (width 0) (type default))
+  )
   (wire (pts (xy 99.06 109.22) (xy 128.27 109.22))
     (stroke (width 0) (type default))
@@
     (stroke (width 0) (type default))
   )
+  (wire (pts (xy 20.32 33.02) (xy 26.67 33.02))
+    (stroke (width 0) (type default))
+  )
   (bus (pts (xy 130.81 104.14) (xy 130.81 106.68))
     (stroke (width 0) (type default))
@@
     (stroke (width 0) (type default))
   )
+  (wire (pts (xy 20.32 30.48) (xy 26.67 30.48))
+    (stroke (width 0) (type default))
+  )
   (wire (pts (xy 99.06 152.4) (xy 128.27 152.4))
     (stroke (width 0) (type default))
@@
     (effects (font (size 1.27 1.27)) (justify left bottom))
   )
+  (label "LED23" (at 20.32 35.56 180) (fields_autoplaced)
+    (effects (font (size 1.27 1.27)) (justify right bottom))
+  )
+  (label "LED24" (at 20.32 38.1 180) (fields_autoplaced)
+    (effects (font (size 1.27 1.27)) (justify right bottom))
+  )
   (label "LED10" (at 99.06 96.52 0) (fields_autoplaced)
     (effects (font (size 1.27 1.27)) (justify left bottom))
@@
     (effects (font (size 1.27 1.27)) (justify left bottom))
   )
+  (label "LED21" (at 20.32 33.02 180) (fields_autoplaced)
+    (effects (font (size 1.27 1.27)) (justify right bottom))
+  )
   (label "LED8" (at 99.06 58.42 0) (fields_autoplaced)
     (effects (font (size 1.27 1.27)) (justify left bottom))
@@
     (effects (font (size 1.27 1.27)) (justify left bottom))
   )
+  (label "LED20" (at 20.32 30.48 180) (fields_autoplaced)
+    (effects (font (size 1.27 1.27)) (justify right bottom))
+  )
   (label "LED6" (at 99.06 53.34 0) (fields_autoplaced)

Commit message: Final routing
Connections:
- net +5V: now also U201.9 (~{MR}), U202.9 (~{MR}), U203.9 (~{MR})
Changed lines of the file:
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@@
+    (stroke (width 0) (type default))
+  )
+  (wire (pts (xy 73.66 147.32) (xy 78.74 147.32))
     (stroke (width 0) (type default))
   )
@@
   )
   (wire (pts (xy 88.9 116.84) (xy 88.9 118.11))
+    (stroke (width 0) (type default))
+  )
+  (wire (pts (xy 73.66 96.52) (xy 78.74 96.52))
+    (stroke (width 0) (type default))
+  )
+  (wire (pts (xy 73.66 43.18) (xy 78.74 43.18))
     (stroke (width 0) (type default))
   )
@@
     (effects (font (size 1.27 1.27)) (justify right))
   )
+  (symbol (lib_id "power:+5V") (at 73.66 147.32 90) (unit 1)
+    (in_bom yes) (on_board yes) (dnp no) (fields_autoplaced)
+    (property "Reference" "#PWR0211" (at 77.47 147.32 0)
+      (effects (font (size 1.27 1.27)) hide)
+    )
+    (property "Value" "+5V" (at 69.85 147.32 90)
+      (effects (font (size 1.27 1.27)) (justify left))
+    )
+    (property "Footprint" "" (at 73.66 147.32 0)
+      (effects (font (size 1.27 1.27)) hide)
+    )
+    (property "Datasheet" "" (at 73.66 147.32 0)
+      (effects (font (size 1.27 1.27)) hide)
+    )
+    (pin "1")
+    (instances
+      (project "LFSR Disc 24"
+        (path "/d11adbca-5bbf-4b99-b4dc-9e7e9b691814/36102b2f-4921-453b-a894-0645b75cde18"
+          (reference "#PWR0211") (unit 1)
+        )
+      )
+    )
+  )
   (symbol (lib_id "power:GND") (at 57.15 190.5 0) (unit 1)
     (in_bom yes) (on_board yes) (dnp no) (fields_autoplaced)
@@
         (path "/d11adbca-5bbf-4b99-b4dc-9e7e9b691814/36102b2f-4921-453b-a894-0645b75cde18"
           (reference "#PWR0202") (unit 1)
+        )
+      )
+    )
+  )
+  (symbol (lib_id "power:+5V") (at 73.66 43.18 90) (unit 1)
+    (in_bom yes) (on_board yes) (dnp no) (fields_autoplaced)
+    (property "Reference" "#PWR0210" (at 77.47 43.18 0)
+      (effects (font (size 1.27 1.27)) hide)
+    )
+    (property "Value" "+5V" (at 69.85 43.18 90)
+      (effects (font (size 1.27 1.27)) (justify left))
+    )
+    (property "Footprint" "" (at 73.66 43.18 0)
+      (effects (font (size 1.27 1.27)) hide)
+    )
+    (property "Datasheet" "" (at 73.66 43.18 0)
+      (effects (font (size 1.27 1.27)) hide)
+    )
+    (pin "1")
+    (instances
+      (project "LFSR Disc 24"
+        (path "/d11adbca-5bbf-4b99-b4dc-9e7e9b691814/36102b2f-4921-453b-a894-0645b75cde18"
+          (reference "#PWR0210") (unit 1)
         )
       )
@@
         )
       )
+    )
+  )
+  (symbol (lib_id "power:+5V") (at 73.66 96.52 90) (unit 1)
+    (in_bom yes) (on_board yes) (dnp no) (fields_autoplaced)
+    (property "Reference" "#PWR0209" (at 77.47 96.52 0)
+      (effects (font (size 1.27 1.27)) hide)
+    )
+    (property "Value" "+5V" (at 69.85 96.52 90)
+      (effects (font (size 1.27 1.27)) (justify left))
+    )
+    (property "Footprint" "" (at 73.66 96.52 0)
+      (effects (font (size 1.27 1.27)) hide)
+    )
+    (property "Datasheet" "" (at 73.66 96.52 0)
+      (effects (font (size 1.27 1.27)) hide)
+    )
+    (pin "1")
+    (instances
+      (project "LFSR Disc 24"
+        (path "/d11adbca-5bbf-4b99-b4dc-9e7e9b691814/36102b2f-4921-453b-a894-0645b75cde18"
+          (reference "#PWR0209") (unit 1)
+        )
+      )
