File: LFSR Disc 24/LFSR Disc 24.kicad_sch (KiCad schematic)
At the start: 0 parts

Commit message: Filling things out a little
Other:
- added sheet Shift Clock (shiftclock.kicad_sch)
- sheet Shift Registers ports: added CLK; removed none
Changed lines of the file:
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@@
     (stroke (width 0) (type default))
+  )
+  (wire (pts (xy 57.15 60.96) (xy 97.79 60.96))
+    (stroke (width 0) (type default))
+  )
+  (sheet (at 34.29 52.07) (size 22.86 19.05) (fields_autoplaced)
+    (stroke (width 0.1524) (type solid))
+    (fill (color 0 0 0 0.0000))
+    (property "Sheetname" "Shift Clock" (at 34.29 51.3584 0)
+      (effects (font (size 1.27 1.27)) (justify left bottom))
+    )
+    (property "Sheetfile" "shiftclock.kicad_sch" (at 34.29 71.7046 0)
+      (effects (font (size 1.27 1.27)) (justify left top))
+    )
+    (pin "CLK" output (at 57.15 60.96 0)
+      (effects (font (size 1.27 1.27)) (justify right))
+    )
+    (instances
+      (project "LFSR Disc 24"
+        (path "/d11adbca-5bbf-4b99-b4dc-9e7e9b691814" (page "4"))
+      )
+    )
   )
   (sheet (at 180.34 52.07) (size 46.99 59.69) (fields_autoplaced)
@@
       (effects (font (size 1.27 1.27)) (justify right))
     )
+    (pin "CLK" input (at 97.79 60.96 180)
+      (effects (font (size 1.27 1.27)) (justify left))
+    )
     (instances

Commit message: Final routing
Parts:
- added J101: USB_A, Connector_USB:USB_A_Molex_67643_Horizontal, symbol Connector:USB_A
- added J102: Conn_01x02_Pin, Connector_PinHeader_2.54mm:PinHeader_1x02_P2.54mm_Vertical, symbol Connector:Conn_01x02_Pin
Connections:
- new net: J101.2 (D-), J101.3 (D+)
- new net +5V: J101.1 (VBUS), J102.2 (Pin_2)
- new net GND: J101.4 (GND), J102.1 (Pin_1)
- no-connect marks 0 -> 1

Commit message: Holes, silkscreen....
Parts:
- added H101, H102, H103, H104: MountingHole, MountingHole:MountingHole_2.7mm_M2.5_ISO7380, symbol Mechanical:MountingHole
Changed lines of the file:
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@@
     (stroke (width 0) (type default))
+  )
+  (symbol (lib_id "Mechanical:MountingHole") (at 95.25 146.05 0) (unit 1)
+    (in_bom yes) (on_board yes) (dnp no) (fields_autoplaced)
+    (property "Reference" "H101" (at 97.79 144.78 0)
+      (effects (font (size 1.27 1.27)) (justify left))
+    )
+    (property "Value" "MountingHole" (at 97.79 147.32 0)
+      (effects (font (size 1.27 1.27)) (justify left))
+    )
+    (property "Footprint" "MountingHole:MountingHole_2.7mm_M2.5_ISO7380" (at 95.25 146.05 0)
+      (effects (font (size 1.27 1.27)) hide)
+    )
+    (property "Datasheet" "~" (at 95.25 146.05 0)
+      (effects (font (size 1.27 1.27)) hide)
+    )
+    (instances
+      (project "LFSR Disc 24"
+        (path "/d11adbca-5bbf-4b99-b4dc-9e7e9b691814"
+          (reference "H101") (unit 1)
+        )
+      )
+    )
   )
   (symbol (lib_id "power:PWR_FLAG") (at 45.72 133.35 180) (unit 1)
@@
     )
   )
+  (symbol (lib_id "Mechanical:MountingHole") (at 95.25 152.4 0) (unit 1)
+    (in_bom yes) (on_board yes) (dnp no) (fields_autoplaced)
+    (property "Reference" "H102" (at 97.79 151.13 0)
+      (effects (font (size 1.27 1.27)) (justify left))
+    )
+    (property "Value" "MountingHole" (at 97.79 153.67 0)
+      (effects (font (size 1.27 1.27)) (justify left))
+    )
+    (property "Footprint" "MountingHole:MountingHole_2.7mm_M2.5_ISO7380" (at 95.25 152.4 0)
+      (effects (font (size 1.27 1.27)) hide)
+    )
+    (property "Datasheet" "~" (at 95.25 152.4 0)
+      (effects (font (size 1.27 1.27)) hide)
+    )
+    (instances
+      (project "LFSR Disc 24"
+        (path "/d11adbca-5bbf-4b99-b4dc-9e7e9b691814"
+          (reference "H102") (unit 1)
+        )
+      )
+    )
+  )
+  (symbol (lib_id "Mechanical:MountingHole") (at 114.3 152.4 0) (unit 1)
+    (in_bom yes) (on_board yes) (dnp no) (fields_autoplaced)
+    (property "Reference" "H104" (at 116.84 151.13 0)
+      (effects (font (size 1.27 1.27)) (justify left))
+    )
+    (property "Value" "MountingHole" (at 116.84 153.67 0)
+      (effects (font (size 1.27 1.27)) (justify left))
+    )
+    (property "Footprint" "MountingHole:MountingHole_2.7mm_M2.5_ISO7380" (at 114.3 152.4 0)
+      (effects (font (size 1.27 1.27)) hide)
+    )
+    (property "Datasheet" "~" (at 114.3 152.4 0)
+      (effects (font (size 1.27 1.27)) hide)
+    )
+    (instances
+      (project "LFSR Disc 24"
+        (path "/d11adbca-5bbf-4b99-b4dc-9e7e9b691814"
+          (reference "H104") (unit 1)
+        )
+      )
+    )
+  )
   (symbol (lib_id "Connector:Conn_01x02_Pin") (at 68.58 124.46 180) (unit 1)
     (in_bom yes) (on_board yes) (dnp no) (fields_autoplaced)
@@
         )
       )
+    )
+  )
+  (symbol (lib_id "Mechanical:MountingHole") (at 114.3 146.05 0) (unit 1)
+    (in_bom yes) (on_board yes) (dnp no) (fields_autoplaced)
+    (property "Reference" "H103" (at 116.84 144.78 0)
+      (effects (font (size 1.27 1.27)) (justify left))
+    )
+    (property "Value" "MountingHole" (at 116.84 147.32 0)
+      (effects (font (size 1.27 1.27)) (justify left))
+    )
+    (property "Footprint" "MountingHole:MountingHole_2.7mm_M2.5_ISO7380" (at 114.3 146.05 0)
+      (effects (font (size 1.27 1.27)) hide)
+    )
+    (property "Datasheet" "~" (at 114.3 146.05 0)
+      (effects (font (size 1.27 1.27)) hide)
+    )
+    (instances
+      (project "LFSR Disc 24"
+        (path "/d11adbca-5bbf-4b99-b4dc-9e7e9b691814"
+          (reference "H103") (unit 1)
+        )
+      )
