File: Two Bit Comparator/Two Bit Comparator.kicad_pcb (KiCad board)
At the start: 2 copper layers, 254 x 203.2 mm, 19 parts, among them U201 74HC00, U202 74HC00, U203 74HC00

Commit message: Starting on accumulation/output stage
Parts:
- added D101: LED, LED_THT:LED_D5.0mm, F.Cu at (243.8, 91.4)
- added D102: LED, LED_THT:LED_D5.0mm, F.Cu at (243.8, 101.6)
- added D103: LED, LED_THT:LED_D5.0mm, F.Cu at (243.8, 111.8)
- added D301: LED, LED_THT:LED_D3.0mm, F.Cu at (157.5, 68.6)
- added D302: LED, LED_THT:LED_D3.0mm, F.Cu at (154.9, 81.3)
- added D303: LED, LED_THT:LED_D3.0mm, F.Cu at (162.6, 78.7)
- added D304: LED, LED_THT:LED_D3.0mm, F.Cu at (172.7, 73.7)
- added D305: LED, LED_THT:LED_D3.0mm, F.Cu at (139.7, 109.2)
- added D306: LED, LED_THT:LED_D3.0mm, F.Cu at (167.6, 109.2)
- added D307: LED, LED_THT:LED_D3.0mm, F.Cu at (173.7, 109.2)
- added D308: LED, LED_THT:LED_D3.0mm, F.Cu at (173.7, 103.7)
- added R101: R, Resistor_THT:R_Axial_DIN0207_L6.3mm_D2.5mm_P7.62mm_Horizontal, F.Cu at (227.3, 91.4)
- added R102: R, Resistor_THT:R_Axial_DIN0207_L6.3mm_D2.5mm_P7.62mm_Horizontal, F.Cu at (227.3, 101.6)
- added R103: R, Resistor_THT:R_Axial_DIN0207_L6.3mm_D2.5mm_P7.62mm_Horizontal, F.Cu at (227.3, 111.8)
- added R301: R, Resistor_THT:R_Axial_DIN0207_L6.3mm_D2.5mm_P7.62mm_Horizontal, F.Cu at (149.9, 72.4)
- added R302: R, Resistor_THT:R_Axial_DIN0207_L6.3mm_D2.5mm_P7.62mm_Horizontal, F.Cu at (131.6, 81.3)
- added R303: R, Resistor_THT:R_Axial_DIN0207_L6.3mm_D2.5mm_P7.62mm_Horizontal, F.Cu at (135.7, 81.3)
- added R304: R, Resistor_THT:R_Axial_DIN0207_L6.3mm_D2.5mm_P7.62mm_Horizontal, F.Cu at (139.7, 81.3)
- added R305: R, Resistor_THT:R_Axial_DIN0207_L6.3mm_D2.5mm_P7.62mm_Horizontal, F.Cu at (147.9, 106.7)
- added R306: R, Resistor_THT:R_Axial_DIN0207_L6.3mm_D2.5mm_P7.62mm_Horizontal, F.Cu at (151.9, 106.7)
- added R307: R, Resistor_THT:R_Axial_DIN0207_L6.3mm_D2.5mm_P7.62mm_Horizontal, F.Cu at (156.0, 106.7)
- added R308: R, Resistor_THT:R_Axial_DIN0207_L6.3mm_D2.5mm_P7.62mm_Horizontal, F.Cu at (160.0, 106.7)
- added U301: 74HC10, Package_DIP:DIP-14_W7.62mm_Socket, F.Cu at (114.3, 177.8)
- added U302: 74HC10, Package_DIP:DIP-14_W7.62mm_Socket, F.Cu at (129.5, 177.8)
- added U303: 74HC10, Package_DIP:DIP-14_W7.62mm_Socket, F.Cu at (144.8, 177.8)
- added U304: 74HC08, Package_DIP:DIP-14_W7.62mm_Socket, F.Cu at (172.7, 177.8)
- added U305: 74HC08, Package_DIP:DIP-14_W7.62mm_Socket, F.Cu at (190.5, 177.8)
- moved U201 25.5 mm to (45.7, 177.8)
- moved U202 25.5 mm to (66.0, 177.8)
- moved U203 25.5 mm to (86.4, 177.8)
- moved D201 25.4 mm to (61.6, 50.8)
- moved D205 25.4 mm to (83.8, 63.5)
- moved D207 25.4 mm to (105.4, 50.8)
- moved R201 25.4 mm to (47.0, 54.6)
- moved R203 25.4 mm to (68.6, 41.9)
- moved R207 25.4 mm to (91.4, 54.6)
- moved D203 25.4 mm to (83.8, 38.1)
- moved R205 25.4 mm to (68.6, 67.3)
Connections:
- net /Compare/A0 renamed /Accumulate and Output/A0
- net /Compare/A1 renamed /Accumulate and Output/A1
- net /Compare/A_{0}NANDB_{0} renamed /Accumulate and Output/A_{0}NANDB_{0}
- net /Compare/A_{0}XNORB_{0} renamed /Accumulate and Output/A_{0}XNORB_{0}
- net /Compare/A_{1}NANDB_{1} renamed /Accumulate and Output/A_{1}NANDB_{1}
- net /Compare/A_{1}XNORB_{1} renamed /Accumulate and Output/A_{1}XNORB_{1}
- net /Compare/B0 renamed /Accumulate and Output/B0
- net /Compare/B1 renamed /Accumulate and Output/B1

Commit message: Thinking about the layout
Parts:
- moved R301 43.7 mm to (130.8, 33.0), turned to 0 degrees
- moved R305 42.0 mm to (121.9, 139.7), turned to 0 degrees
- moved D302 41.9 mm to (144.8, 40.6)
- moved R302 40.6 mm to (130.8, 40.6), turned to 0 degrees
- moved D307 39.6 mm to (137.2, 124.5)
- moved R308 39.4 mm to (121.9, 116.8), turned to 0 degrees
- moved R306 39.3 mm to (121.9, 132.1), turned to 0 degrees
- moved D308 38.8 mm to (137.2, 116.8)
- moved R307 38.4 mm to (121.9, 124.5), turned to 0 degrees
- moved D306 38.1 mm to (137.2, 132.1)
- moved D301 37.8 mm to (144.8, 33.0)
- moved D303 35.3 mm to (144.8, 48.3)
- moved R303 33.4 mm to (130.8, 48.3), turned to 0 degrees
- moved D304 33.1 mm to (144.8, 55.9)
- moved R103 31.4 mm to (234.9, 142.2)
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Connections:
- U301 pad 1: unconnected-(U301-Pad1) -> /Accumulate and Output/B1
- U301 pad 2: unconnected-(U301-Pad2) -> /Accumulate and Output/A_{1}NANDB_{1}
- U301 pad 3: unconnected-(U301-Pad3) -> /Accumulate and Output/A_{1}NANDB_{1}
- U301 pad 4: unconnected-(U301-Pad4) -> /Accumulate and Output/A1
- U302 pad 1: unconnected-(U302-Pad1) -> /Accumulate and Output/B0
- U302 pad 10: unconnected-(U302-Pad10) -> /Accumulate and Output/A_{0}XNORB_{0}
- U302 pad 11: unconnected-(U302-Pad11) -> /Accumulate and Output/I_{A=B}
- U302 pad 13: unconnected-(U302-Pad13) -> /Accumulate and Output/A_{1}XNORB_{1}
- U302 pad 2: unconnected-(U302-Pad2) -> /Accumulate and Output/A_{0}NANDB_{0}
- U302 pad 3: unconnected-(U302-Pad3) -> /Accumulate and Output/A_{1}XNORB_{1}
- U302 pad 4: unconnected-(U302-Pad4) -> /Accumulate and Output/A_{0}XNORB_{0}
- U302 pad 5: unconnected-(U302-Pad5) -> /Accumulate and Output/I_{A<B}
- U302 pad 9: unconnected-(U302-Pad9) -> /Accumulate and Output/A_{1}XNORB_{1}
- U303 pad 1: unconnected-(U303-Pad1) -> /Accumulate and Output/A_{1}XNORB_{1}
- U303 pad 10: unconnected-(U303-Pad10) -> /Accumulate and Output/A_{0}NANDB_{0}
- U303 pad 11: unconnected-(U303-Pad11) -> /Accumulate and Output/A0
- U303 pad 13: unconnected-(U303-Pad13) -> /Accumulate and Output/I_{A=B}
- U303 pad 2: unconnected-(U303-Pad2) -> /Accumulate and Output/A_{0}XNORB_{0}
- U303 pad 3: unconnected-(U303-Pad3) -> /Accumulate and Output/I_{A>B}
- U303 pad 4: unconnected-(U303-Pad4) -> /Accumulate and Output/A_{1}XNORB_{1}
- U303 pad 5: unconnected-(U303-Pad5) -> /Accumulate and Output/A_{0}XNORB_{0}
- U303 pad 9: unconnected-(U303-Pad9) -> /Accumulate and Output/A_{1}XNORB_{1}
Other:
- board size 254 x 203.2 mm -> 254 x 215.9 mm
- board text added: "A0"
- board text added: "A1"
- board text added: "A_{1} = B_{1}"
- board text added: "A_{1} AND ( A_{1} NAND B_{1} )"
- board text added: "B0"
- board text added: "B0 AND ( A0 NAND B0 ) AND ( A1 XNOR B1 )"
- board text added: "B1"
- board text added: "B1 AND ( A1 NAND B1 )"
- board text added: "B_{0} AND ( A_{0} NAND B_{0} ) AND ( A_{1} = B_{1} )"
- board text added: "I_{A < B} AND ( A0 XNOR B0 ) AND ( A1 XNOR B1 )"
- board text added: "I_{A = B} AND ( A0 XNOR B0 ) AND ( A1 XNOR B1 )"
- board text added: "I_{A = B} AND ( A_{0} = B_{0} ) AND ( A_{1} = B_{1} )"
- board text added: "I_{A > B} AND ( A_{0} = B_{0} ) AND ( A_{1} = B_{1} )"
- board text added: "If none of the following are true"
- board text added: "then O_{A < B}"
- board text added: "then O_{A > B}"
