File: Two Bit Comparator/accandout.kicad_sch (KiCad schematic)
At the start: 21 parts, among them U301 74HC10, U302 74HC10, U303 74HC10, U304 74HC08, U305 74HC08

Commit message: Thinking about the layout
Connections:
- net A_{0}NANDB_{0}: now also U302.2, U303.10
- net A_{0}XNORB_{0}: now also U302.10, U302.4, U303.2, U303.5
- net A_{1}NANDB_{1}: now also U301.2, U301.3
- net A_{1}XNORB_{1}: now also U302.13, U302.3, U302.9, U303.1, U303.4, U303.9
- net I_{A<B}: now also U302.5
- net I_{A=B}: now also U302.11, U303.13
- net I_{A>B}: now also U303.3
- net B1: now reaches U301.1
- net A1: now reaches U301.4
- net B0: now reaches U302.1
- net A0: now reaches U303.11
Other:
- note added: "Note this is a duplicate of the above"
Changed lines of the file:
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@@
   )
   (no_connect (at 223.52 156.21))
+  (wire (pts (xy 41.91 29.21) (xy 48.26 29.21))
+    (stroke (width 0) (type default))
+  )
   (wire (pts (xy 106.68 76.2) (xy 101.6 76.2))
     (stroke (width 0) (type default))
@@
     (stroke (width 0) (type default))
   )
+  (wire (pts (xy 43.18 102.87) (xy 48.26 102.87))
+    (stroke (width 0) (type default))
+  )
+  (wire (pts (xy 43.18 69.85) (xy 48.26 69.85))
+    (stroke (width 0) (type default))
+  )
+  (wire (pts (xy 41.91 46.99) (xy 48.26 46.99))
+    (stroke (width 0) (type default))
+  )
   (wire (pts (xy 48.26 31.75) (xy 45.72 31.75))
     (stroke (width 0) (type default))
@@
     (stroke (width 0) (type default))
   )
+  (wire (pts (xy 40.64 26.67) (xy 48.26 26.67))
+    (stroke (width 0) (type default))
+  )
   (wire (pts (xy 200.66 153.67) (xy 207.01 153.67))
     (stroke (width 0) (type default))
@@
     (stroke (width 0) (type default))
   )
+  (wire (pts (xy 43.18 105.41) (xy 48.26 105.41))
+    (stroke (width 0) (type default))
+  )
   (wire (pts (xy 245.11 39.37) (xy 245.11 41.91))
     (stroke (width 0) (type default))
   )
+  (wire (pts (xy 43.18 85.09) (xy 48.26 85.09))
+    (stroke (width 0) (type default))
+  )
   (wire (pts (xy 256.54 39.37) (xy 256.54 41.91))
     (stroke (width 0) (type default))
@@
     (stroke (width 0) (type default))
   )
+  (wire (pts (xy 43.18 123.19) (xy 48.26 123.19))
+    (stroke (width 0) (type default))
+  )
+  (wire (pts (xy 43.18 143.51) (xy 48.26 143.51))
+    (stroke (width 0) (type default))
+  )
   (wire (pts (xy 215.9 29.21) (xy 215.9 31.75))
     (stroke (width 0) (type default))
@@
     (stroke (width 0) (type default))
   )
+  (wire (pts (xy 43.18 64.77) (xy 48.26 64.77))
+    (stroke (width 0) (type default))
+  )
   (wire (pts (xy 245.11 49.53) (xy 245.11 53.34))
     (stroke (width 0) (type default))
@@
     (stroke (width 0) (type default))
   )
+  (wire (pts (xy 43.18 120.65) (xy 48.26 120.65))
+    (stroke (width 0) (type default))
+  )
   (wire (pts (xy 45.72 31.75) (xy 45.72 34.29))
     (stroke (width 0) (type default))
@@
     (stroke (width 0) (type default))
   )
+  (wire (pts (xy 41.91 49.53) (xy 48.26 49.53))
+    (stroke (width 0) (type default))
+  )
+  (wire (pts (xy 43.18 158.75) (xy 48.26 158.75))
+    (stroke (width 0) (type default))
+  )
   (wire (pts (xy 209.55 53.34) (xy 215.9 53.34))
     (stroke (width 0) (type default))
@@
     (stroke (width 0) (type default))
   )
+  (wire (pts (xy 41.91 146.05) (xy 48.26 146.05))
+    (stroke (width 0) (type default))
+  )
+  (wire (pts (xy 43.18 161.29) (xy 48.26 161.29))
+    (stroke (width 0) (type default))
+  )
   (wire (pts (xy 76.2 143.51) (xy 76.2 149.86))
     (stroke (width 0) (type default))
@@
     (stroke (width 0) (type default))
   )
+  (wire (pts (xy 43.18 140.97) (xy 48.26 140.97))
+    (stroke (width 0) (type default))
+  )
   (wire (pts (xy 133.35 99.06) (xy 142.24 99.06))
     (stroke (width 0) (type default))
@@
     (stroke (width 0) (type default))
   )
+  (wire (pts (xy 41.91 44.45) (xy 48.26 44.45))
+    (stroke (width 0) (type default))
+  )
   (wire (pts (xy 203.2 39.37) (xy 203.2 41.91))
     (stroke (width 0) (type default))
   )
+  (wire (pts (xy 43.18 82.55) (xy 48.26 82.55))
+    (stroke (width 0) (type default))
+  )
   (wire (pts (xy 207.01 153.67) (xy 208.28 153.67))
     (stroke (width 0) (type default))
@@
     (stroke (width 0) (type default))
   )
+  (wire (pts (xy 43.18 87.63) (xy 48.26 87.63))
+    (stroke (width 0) (type default))
+  )
   (wire (pts (xy 116.84 165.1) (xy 139.7 165.1))
     (stroke (width 0) (type default))
@@
     (stroke (width 0) (type default))
   )
+  (wire (pts (xy 43.18 125.73) (xy 48.26 125.73))
+    (stroke (width 0) (type default))
+  )
   (wire (pts (xy 63.5 143.51) (xy 76.2 143.51))
     (stroke (width 0) (type default))
@@
     (stroke (width 0) (type default))
   )
+  (wire (pts (xy 43.18 67.31) (xy 48.26 67.31))
+    (stroke (width 0) (type default))
+  )
   (wire (pts (xy 106.68 54.61) (xy 111.76 54.61))
     (stroke (width 0) (type default))
@@
     (stroke (width 0) (type default))
   )
+  (wire (pts (xy 43.18 107.95) (xy 48.26 107.95))
+    (stroke (width 0) (type default))
+  )
   (wire (pts (xy 76.2 154.94) (xy 76.2 161.29))
     (stroke (width 0) (type default))
@@
     (stroke (width 0) (type default))
   )
+  (text "Note this is a duplicate\nof the above" (at 59.69 101.6 0)
+    (effects (font (size 1.27 1.27)) (justify left bottom))
+  )
   (label "c1" (at 76.2 46.99 0) (fields_autoplaced)
     (effects (font (size 1.27 1.27)) (justify left bottom))
@@
     (effects (font (size 1.27 1.27)) (justify left bottom))
   )
+  (label "B1" (at 40.64 26.67 0) (fields_autoplaced)
+    (effects (font (size 1.27 1.27)) (justify left bottom))
+  )
   (label "c0" (at 180.34 29.21 0) (fields_autoplaced)
     (effects (font (size 1.27 1.27)) (justify left bottom))
   )
+  (label "B0" (at 41.91 44.45 0) (fields_autoplaced)
+    (effects (font (size 1.27 1.27)) (justify left bottom))
+  )
   (label "c6" (at 76.2 143.51 0) (fields_autoplaced)
     (effects (font (size 1.27 1.27)) (justify left bottom))
   )
+  (label "A1" (at 43.18 161.29 0) (fields_autoplaced)
+    (effects (font (size 1.27 1.27)) (justify left bottom))
+  )
   (label "c4" (at 76.2 105.41 0) (fields_autoplaced)
     (effects (font (size 1.27 1.27)) (justify left bottom))
@@
     (effects (font (size 1.27 1.27)) (justify left bottom))
   )
+  (label "A0" (at 41.91 146.05 0) (fields_autoplaced)
+    (effects (font (size 1.27 1.27)) (justify left bottom))
+  )
   (label "c5" (at 245.11 29.21 0) (fields_autoplaced)
     (effects (font (size 1.27 1.27)) (justify left bottom))
@@
   (label "c2" (at 203.2 29.21 0) (fields_autoplaced)
     (effects (font (size 1.27 1.27)) (justify left bottom))
-  )
-  (hierarchical_label "I_{A<B}" (shape input) (at 20.32 78.74 180) (fields_autoplaced)
-    (effects (font (size 1.27 1.27)) (justify right))
   )
   (hierarchical_label "O_{A<B}" (shape output) (at 139.7 133.35 0) (fields_autoplaced)
     (effects (font (size 1.27 1.27)) (justify left))
   )
+  (hierarchical_label "A_{0}XNORB_{0}" (shape input) (at 43.18 67.31 180) (fields_autoplaced)
+    (effects (font (size 1.27 1.27)) (justify right))
+  )
+  (hierarchical_label "I_{A=B}" (shape input) (at 43.18 87.63 180) (fields_autoplaced)
+    (effects (font (size 1.27 1.27)) (justify right))
+  )
+  (hierarchical_label "A_{1}XNORB_{1}" (shape input) (at 43.18 64.77 180) (fields_autoplaced)
+    (effects (font (size 1.27 1.27)) (justify right))
+  )
+  (hierarchical_label "A_{0}XNORB_{0}" (shape input) (at 43.18 125.73 180) (fields_autoplaced)
+    (effects (font (size 1.27 1.27)) (justify right))
+  )
+  (hierarchical_label "A_{0}NANDB_{0}" (shape input) (at 43.18 143.51 180) (fields_autoplaced)
+    (effects (font (size 1.27 1.27)) (justify right))
+  )
+  (hierarchical_label "I_{A<B}" (shape input) (at 43.18 69.85 180) (fields_autoplaced)
+    (effects (font (size 1.27 1.27)) (justify right))
+  )
   (hierarchical_label "A_{0}XNORB_{0}" (shape input) (at 133.35 93.98 180) (fields_autoplaced)
     (effects (font (size 1.27 1.27)) (justify right))
@@
     (effects (font (size 1.27 1.27)) (justify left))
   )
-  (hierarchical_label "A_{1}NANDB_{1}" (shape input) (at 24.13 72.39 180) (fields_autoplaced)
+  (hierarchical_label "A_{1}NANDB_{1}" (shape input) (at 43.18 158.75 180) (fields_autoplaced)
+    (effects (font (size 1.27 1.27)) (justify right))
+  )
+  (hierarchical_label "I_{A>B}" (shape input) (at 43.18 120.65 180) (fields_autoplaced)
+    (effects (font (size 1.27 1.27)) (justify right))
+  )
+  (hierarchical_label "A_{1}XNORB_{1}" (shape input) (at 43.18 82.55 180) (fields_autoplaced)
     (effects (font (size 1.27 1.27)) (justify right))
   )
@@
     (effects (font (size 1.27 1.27)) (justify right))
   )
-  (hierarchical_label "A_{0}NANDB_{0}" (shape input) (at 25.4 101.6 180) (fields_autoplaced)
-    (effects (font (size 1.27 1.27)) (justify right))
-  )
   (hierarchical_label "B[0..1]" (shape input) (at 21.59 96.52 180) (fields_autoplaced)
     (effects (font (size 1.27 1.27)) (justify right))
   )
+  (hierarchical_label "A_{1}XNORB_{1}" (shape input) (at 43.18 102.87 180) (fields_autoplaced)
+    (effects (font (size 1.27 1.27)) (justify right))
+  )
+  (hierarchical_label "A_{1}NANDB_{1}" (shape input) (at 41.91 29.21 180) (fields_autoplaced)
+    (effects (font (size 1.27 1.27)) (justify right))
+  )
+  (hierarchical_label "A_{1}XNORB_{1}" (shape input) (at 41.91 49.53 180) (fields_autoplaced)
+    (effects (font (size 1.27 1.27)) (justify right))
+  )
+  (hierarchical_label "A_{0}XNORB_{0}" (shape input) (at 43.18 85.09 180) (fields_autoplaced)
+    (effects (font (size 1.27 1.27)) (justify right))
+  )
   (hierarchical_label "I_{A=B}" (shape input) (at 133.35 101.6 180) (fields_autoplaced)
     (effects (font (size 1.27 1.27)) (justify right))
@@
     (effects (font (size 1.27 1.27)) (justify right))
   )
-  (hierarchical_label "I_{A>B}" (shape input) (at 21.59 115.57 180) (fields_autoplaced)
-    (effects (font (size 1.27 1.27)) (justify right))
-  )
+  (hierarchical_label "A_{0}NANDB_{0}" (shape input) (at 41.91 46.99 180) (fields_autoplaced)
+    (effects (font (size 1.27 1.27)) (justify right))
+  )
+  (hierarchical_label "A_{1}XNORB_{1}" (shape input) (at 43.18 140.97 180) (fields_autoplaced)
+    (effects (font (size 1.27 1.27)) (justify right))
+  )
+  (hierarchical_label "I_{A=B}" (shape input) (at 43.18 107.95 180) (fields_autoplaced)
+    (effects (font (size 1.27 1.27)) (justify right))
+  )
+  (hierarchical_label "A_{1}XNORB_{1}" (shape input) (at 43.18 123.19 180) (fields_autoplaced)
+    (effects (font (size 1.27 1.27)) (justify right))
+  )
+  (hierarchical_label "A_{0}XNORB_{0}" (shape input) (at 43.18 105.41 180) (fields_autoplaced)
+    (effects (font (size 1.27 1.27)) (justify right))
+  )
