File: Runner 4017/Runner 4017.kicad_sch (KiCad schematic)
At the start: 23 parts, among them U101 4017

Commit message: Working through things
Parts:
- added C101: 10u, Capacitor_THT:CP_Radial_D4.0mm_P1.50mm, symbol Device:C_Polarized
- added H101, H102, H103, H104: MountingHole, MountingHole:MountingHole_2.7mm_M2.5_ISO7380, symbol Mechanical:MountingHole
- added J101: USB_A, Connector_USB:USB_A_Molex_67643_Horizontal, symbol Connector:USB_A
- added J102: Conn_01x02_Pin, Connector_PinHeader_2.54mm:PinHeader_1x02_P2.54mm_Vertical, symbol Connector:Conn_01x02_Pin
- added R107: 1k, Resistor_THT:R_Axial_DIN0207_L6.3mm_D2.5mm_P7.62mm_Horizontal, symbol Device:R
- added R108: 100k, Resistor_THT:R_Axial_DIN0207_L6.3mm_D2.5mm_P7.62mm_Horizontal, symbol Device:R
Connections:
- net +5V: now also C101.1, J101.1 (VBUS), J102.2 (Pin_2), R108.1
- net GND: now also J101.4 (GND), J102.1 (Pin_1), R107.1
- net RESET: now reaches U101.15 (Reset)
- net RESET: now also C101.2, R107.2, R108.2
- new net: J101.2 (D-), J101.3 (D+)
- no-connect marks 1 -> 2
