File: Runner 4017/Runner 4017.kicad_pcb (KiCad board)
At the start: 2 copper layers, 23 parts, among them U101 4017

Commit message: Working through things
Parts:
- added C101: 10u, Capacitor_THT:CP_Radial_D4.0mm_P1.50mm, F.Cu at (110.7, 83.8)
- added C201: 10u, Capacitor_THT:CP_Radial_D4.0mm_P1.50mm, F.Cu at (109.2, 109.2)
- added C202: 0.1u, Capacitor_THT:C_Disc_D4.3mm_W1.9mm_P5.00mm, F.Cu at (116.8, 87.6)
- added C203: 0.01u, Capacitor_THT:C_Disc_D3.4mm_W2.1mm_P2.50mm, F.Cu at (116.8, 109.3)
- added H101: MountingHole, MountingHole:MountingHole_2.7mm_M2.5_ISO7380, F.Cu at (94.0, 50.8)
- added H102: MountingHole, MountingHole:MountingHole_2.7mm_M2.5_ISO7380, F.Cu at (152.4, 50.8)
- added H103: MountingHole, MountingHole:MountingHole_2.7mm_M2.5_ISO7380, F.Cu at (94.0, 116.8)
- added H104: MountingHole, MountingHole:MountingHole_2.7mm_M2.5_ISO7380, F.Cu at (152.4, 116.8)
- added J101: USB_A, Connector_USB:USB_A_Molex_67643_Horizontal, F.Cu at (101.6, 63.5)
- added J102: Conn_01x02_Pin, Connector_PinHeader_2.54mm:PinHeader_1x02_P2.54mm_Vertical, F.Cu at (91.4, 81.3)
- added R107: 1k, Resistor_THT:R_Axial_DIN0207_L6.3mm_D2.5mm_P7.62mm_Horizontal, F.Cu at (96.5, 81.3)
- added R108: 100k, Resistor_THT:R_Axial_DIN0207_L6.3mm_D2.5mm_P7.62mm_Horizontal, F.Cu at (96.5, 86.4)
- added R201: 10k, Resistor_THT:R_Axial_DIN0207_L6.3mm_D2.5mm_P7.62mm_Horizontal, F.Cu at (104.1, 96.5)
- added R202: 22k, Resistor_THT:R_Axial_DIN0207_L6.3mm_D2.5mm_P7.62mm_Horizontal, F.Cu at (104.1, 101.6)
- added R203: 1k, Resistor_THT:R_Axial_DIN0207_L6.3mm_D2.5mm_P7.62mm_Horizontal, F.Cu at (104.1, 106.7)
- added U201: LM555xN, Package_DIP:DIP-8_W7.62mm_Socket, F.Cu at (109.2, 96.5)
- moved U101 17.8 mm to (109.2, 58.4)
Connections:
- U101 pad 14: unconnected-(U101-CLK-Pad14) -> /Clock/CLK
- U101 pad 15: unconnected-(U101-Reset-Pad15) -> /RESET
Routing:
- net Net-(D106-A): track 0.00 -> 67.1 mm
- net /Clock/CLK: track 0.00 -> 54.4 mm
- net /Clock/TRTHR: track 0.00 -> 48.9 mm
- net Net-(D107-A): track 0.00 -> 20.6 mm
- net /Clock/DIVIDER: track 0.00 -> 19.2 mm
- net Net-(D105-A): track 0.00 -> 14.9 mm
- net unconnected-(J101-Shield-Pad5): track 0.00 -> 13.1 mm
- net /RESET: track 0.00 -> 11.2 mm
- net Net-(D108-A): track 0.00 -> 9.15 mm
- net /LED5: track 0.00 -> 7.18 mm
- net /LED4: track 0.00 -> 7.18 mm
- net /LED3: track 0.00 -> 7.18 mm
- net /LED2: track 0.00 -> 7.18 mm
- net Net-(U201-CV): track 0.00 -> 5.12 mm
- net Net-(D116-A): track 0.00 -> 5.08 mm
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Other:
- board outline added: 68.6 x 76.2 mm
- board text added: "RGE2023"
- board text added: "Running 4017"

Commit message: Zone fills
Routing:
- net /RESET: track 11.2 -> 43.5 mm
- net Net-(D104-A): track 0.00 -> 29.4 mm, vias 0 -> 1
- net Net-(D107-A): track 20.6 -> 49.7 mm, vias 0 -> 1
- net Net-(D108-A): track 9.15 -> 37.0 mm, vias 0 -> 1
- net Net-(D103-A): track 0.00 -> 26.8 mm, vias 0 -> 1
- net Net-(D101-A): track 0.00 -> 24.3 mm, vias 0 -> 1
- net Net-(D102-A): track 0.00 -> 21.7 mm, vias 0 -> 1
- net Net-(D105-A): track 14.9 -> 32.6 mm, vias 0 -> 1
- net Net-(D109-A): track 0.00 -> 14.5 mm, vias 0 -> 1
- net Net-(D110-A): track 0.00 -> 10.2 mm
- added copper zone on B.Cu, net +5V
- added copper zone on F.Cu, net GND
Other:
- board text added: "+5V"
- board text added: "GND"
Changed lines of the file:
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@@
     (effects (font (size 1.6256 1.6256) (thickness 0.2032)) (justify left bottom mirror))
+  )
+  (gr_text "+5V" (at 93.98 83.82) (layer "F.SilkS")
+    (effects (font (size 0.8128 0.8128) (thickness 0.1524)))
+  )
+  (gr_text "GND" (at 93.98 81.28) (layer "F.SilkS")
+    (effects (font (size 0.8128 0.8128) (thickness 0.1524)))
   )
   (gr_text "Running 4017" (at 101.6 53.34) (layer "F.SilkS")
@@
   )
   (segment (start 134.62 58.42) (end 137.16 58.42) (width 0.127) (layer "F.Cu") (net 1))
+  (segment (start 121.92 59.055) (end 121.92 64.77) (width 0.127) (layer "F.Cu") (net 2))
+  (segment (start 127 58.42) (end 122.555 58.42) (width 0.127) (layer "F.Cu") (net 2))
+  (segment (start 122.555 58.42) (end 121.92 59.055) (width 0.127) (layer "F.Cu") (net 2))
+  (via (at 121.92 64.77) (size 0.499999) (drill 0.20066) (layers "F.Cu" "B.Cu") (net 2))
+  (segment (start 110.49 64.77) (end 109.22 63.5) (width 0.127) (layer "B.Cu") (net 2))
+  (segment (start 121.92 64.77) (end 110.49 64.77) (width 0.127) (layer "B.Cu") (net 2))
   (segment (start 137.16 68.58) (end 134.62 71.12) (width 0.127) (layer "F.Cu") (net 3))
   (segment (start 134.62 66.04) (end 137.16 68.58) (width 0.127) (layer "F.Cu") (net 3))
+  (segment (start 121.92 66.04) (end 121.285 65.405) (width 0.127) (layer "F.Cu") (net 4))
+  (segment (start 121.285 65.405) (end 121.285 62.23) (width 0.127) (layer "F.Cu") (net 4))
+  (segment (start 127 66.04) (end 121.92 66.04) (width 0.127) (layer "F.Cu") (net 4))
+  (via (at 121.285 62.23) (size 0.499999) (drill 0.20066) (layers "F.Cu" "B.Cu") (net 4))
+  (segment (start 121.285 62.23) (end 110.49 62.23) (width 0.127) (layer "B.Cu") (net 4))
+  (segment (start 110.49 62.23) (end 109.22 60.96) (width 0.127) (layer "B.Cu") (net 4))
   (segment (start 134.62 76.2) (end 137.16 78.74) (width 0.127) (layer "F.Cu") (net 5))
   (segment (start 137.16 78.74) (end 134.62 81.28) (width 0.127) (layer "F.Cu") (net 5))
+  (segment (start 127 76.2) (end 124.46 76.2) (width 0.127) (layer "F.Cu") (net 6))
+  (segment (start 123.825 75.565) (end 123.825 67.31) (width 0.127) (layer "F.Cu") (net 6))
+  (segment (start 124.46 76.2) (end 123.825 75.565) (width 0.127) (layer "F.Cu") (net 6))
+  (via (at 123.825 67.31) (size 0.499999) (drill 0.20066) (layers "F.Cu" "B.Cu") (net 6))
+  (segment (start 110.49 67.31) (end 109.22 66.04) (width 0.127) (layer "B.Cu") (net 6))
+  (segment (start 123.825 67.31) (end 110.49 67.31) (width 0.127) (layer "B.Cu") (net 6))
   (segment (start 134.62 86.36) (end 137.16 88.9) (width 0.127) (layer "F.Cu") (net 7))
   (segment (start 134.62 91.44) (end 137.16 88.9) (width 0.127) (layer "F.Cu") (net 7))
+  (segment (start 127 86.36) (end 123.825 86.36) (width 0.127) (layer "F.Cu") (net 8))
+  (segment (start 123.825 86.36) (end 123.19 85.725) (width 0.127) (layer "F.Cu") (net 8))
+  (segment (start 123.19 85.725) (end 123.19 74.93) (width 0.127) (layer "F.Cu") (net 8))
+  (via (at 123.19 74.93) (size 0.499999) (drill 0.20066) (layers "F.Cu" "B.Cu") (net 8))
+  (segment (start 110.49 74.93) (end 109.22 73.66) (width 0.127) (layer "B.Cu") (net 8))
+  (segment (start 123.19 74.93) (end 110.49 74.93) (width 0.127) (layer "B.Cu") (net 8))
   (segment (start 137.16 99.06) (end 134.62 101.6) (width 0.127) (layer "F.Cu") (net 9))
   (segment (start 134.62 96.52) (end 137.16 99.06) (width 0.127) (layer "F.Cu") (net 9))
   (segment (start 127 96.52) (end 122.555 96.52) (width 0.127) (layer "F.Cu") (net 10))
   (segment (start 121.92 95.885) (end 121.92 86.36) (width 0.127) (layer "F.Cu") (net 10))
+  (segment (start 121.92 86.36) (end 121.92 73.66) (width 0.127) (layer "F.Cu") (net 10))
   (segment (start 122.555 96.52) (end 121.92 95.885) (width 0.127) (layer "F.Cu") (net 10))
+  (via (at 121.92 73.66) (size 0.499999) (drill 0.20066) (layers "F.Cu" "B.Cu") (net 10))
+  (segment (start 121.92 73.66) (end 116.84 73.66) (width 0.127) (layer "B.Cu") (net 10))
   (segment (start 137.16 109.22) (end 134.62 109.22) (width 0.127) (layer "F.Cu") (net 11))
   (segment (start 121.285 109.22) (end 120.65 108.585) (width 0.127) (layer "F.Cu") (net 12))
@@
   (segment (start 127 109.22) (end 121.285 109.22) (width 0.127) (layer "F.Cu") (net 12))
   (segment (start 120.015 59.69) (end 110.49 59.69) (width 0.127) (layer "F.Cu") (net 12))
+  (segment (start 121.285 86.36) (end 121.285 69.85) (width 0.127) (layer "F.Cu") (net 13))
   (segment (start 127 101.6) (end 121.92 101.6) (width 0.127) (layer "F.Cu") (net 13))
   (segment (start 121.285 100.965) (end 121.285 86.36) (width 0.127) (layer "F.Cu") (net 13))
   (segment (start 121.92 101.6) (end 121.285 100.965) (width 0.127) (layer "F.Cu") (net 13))
+  (via (at 121.285 69.85) (size 0.499999) (drill 0.20066) (layers "F.Cu" "B.Cu") (net 13))
+  (segment (start 110.49 69.85) (end 109.22 68.58) (width 0.127) (layer "B.Cu") (net 13))
+  (segment (start 121.285 69.85) (end 110.49 69.85) (width 0.127) (layer "B.Cu") (net 13))
+  (segment (start 122.555 86.36) (end 122.555 72.39) (width 0.127) (layer "F.Cu") (net 14))
   (segment (start 122.555 90.805) (end 122.555 86.36) (width 0.127) (layer "F.Cu") (net 14))
   (segment (start 127 91.44) (end 123.19 91.44) (width 0.127) (layer "F.Cu") (net 14))
   (segment (start 123.19 91.44) (end 122.555 90.805) (width 0.127) (layer "F.Cu") (net 14))
+  (via (at 122.555 72.39) (size 0.499999) (drill 0.20066) (layers "F.Cu" "B.Cu") (net 14))
+  (segment (start 110.49 72.39) (end 109.22 71.12) (width 0.127) (layer "B.Cu") (net 14))
+  (segment (start 122.555 72.39) (end 110.49 72.39) (width 0.127) (layer "B.Cu") (net 14))
+  (segment (start 124.46 81.28) (end 123.825 80.645) (width 0.127) (layer "F.Cu") (net 15))
+  (segment (start 123.825 80.645) (end 123.825 76.835) (width 0.127) (layer "F.Cu") (net 15))
+  (segment (start 127 81.28) (end 124.46 81.28) (width 0.127) (layer "F.Cu") (net 15))
+  (via (at 123.825 76.835) (size 0.499999) (drill 0.20066) (layers "F.Cu" "B.Cu") (net 15))
+  (segment (start 117.475 76.835) (end 116.84 76.2) (width 0.127) (layer "B.Cu") (net 15))
+  (segment (start 123.825 76.835) (end 117.475 76.835) (width 0.127) (layer "B.Cu") (net 15))
+  (segment (start 116.84 71.12) (end 127 71.12) (width 0.127) (layer "B.Cu") (net 16))
   (segment (start 144.78 58.42) (end 149.86 58.42) (width 0.127) (layer "F.Cu") (net 18))
   (segment (start 144.78 68.58) (end 149.86 68.58) (width 0.127) (layer "F.Cu") (net 19))
@@
   (segment (start 144.78 99.06) (end 149.86 99.06) (width 0.127) (layer "F.Cu") (net 22))
   (segment (start 144.78 109.22) (end 149.86 109.22) (width 0.127) (layer "F.Cu") (net 23))
+  (segment (start 112.395 60.96) (end 111.76 61.595) (width 0.127) (layer "F.Cu") (net 25))
+  (segment (start 111.125 81.28) (end 104.14 81.28) (width 0.127) (layer "F.Cu") (net 25))
   (segment (start 104.14 81.28) (end 104.14 86.36) (width 0.127) (layer "F.Cu") (net 25))
   (segment (start 104.14 86.36) (end 106.68 86.36) (width 0.127) (layer "F.Cu") (net 25))
+  (segment (start 111.76 80.645) (end 111.125 81.28) (width 0.127) (layer "F.Cu") (net 25))
+  (segment (start 111.76 61.595) (end 111.76 80.645) (width 0.127) (layer "F.Cu") (net 25))
+  (segment (start 116.84 60.96) (end 112.395 60.96) (width 0.127) (layer "F.Cu") (net 25))
   (segment (start 106.68 86.36) (end 109.22 83.82) (width 0.127) (layer "F.Cu") (net 25))
   (segment (start 114.3 108.585) (end 114.3 102.235) (width 0.127) (layer "F.Cu") (net 26))
@@
   (segment (start 113.665 63.5) (end 113.03 64.135) (width 0.127) (layer "F.Cu") (net 32))
   (segment (start 106.045 102.235) (end 106.68 101.6) (width 0.127) (layer "F.Cu") (net 32))
+  (zone (net 17) (net_name "GND") (layer "F.Cu") (hatch edge 0.508)
+    (connect_pads (clearance 0.254))
+    (min_thickness 0.127) (filled_areas_thickness no)
+    (fill yes (thermal_gap 0.5) (thermal_bridge_width 0.5) (smoothing fillet) (radius 0.127))
+    (polygon
+      (pts
+        (xy 86.36 43.18)
+        (xy 160.02 43.18)
+        (xy 160.02 124.46)
+        (xy 86.36 124.46)
+      )
+    )
+  )
+  (zone (net 27) (net_name "+5V") (layer "B.Cu") (hatch edge 0.508)
+    (priority 1)
+    (connect_pads (clearance 0.254))
+    (min_thickness 0.127) (filled_areas_thickness no)
+    (fill yes (thermal_gap 0.5) (thermal_bridge_width 0.5) (smoothing fillet) (radius 0.127))
+    (polygon
+      (pts
+        (xy 83.82 40.64)
+        (xy 162.56 40.64)
+        (xy 162.56 127)
+        (xy 83.82 127)
+      )
+    )
+  )
 )
