File: Binary Flip Flop Counter/Binary Flip Flop Counter.kicad_sch (KiCad schematic)
At the start: 0 parts

Commit message: Routing quickly
Parts:
- added H101, H102, H103, H104: MountingHole, MountingHole:MountingHole_2.7mm_M2.5_ISO7380, symbol Mechanical:MountingHole
- added J101: USB_A, Connector_USB:USB_A_Molex_67643_Horizontal, symbol Connector:USB_A
- added J102: Conn_01x02_Pin, Connector_PinHeader_2.54mm:PinHeader_1x02_P2.54mm_Vertical, symbol Connector:Conn_01x02_Pin
Connections:
- new net: J101.2 (D-), J101.3 (D+)
- new net +5V: J101.1 (VBUS), J102.2 (Pin_2)
- new net GND: J101.4 (GND), J102.1 (Pin_1)
- no-connect marks 0 -> 1
