File: Binary Flip Flop Counter/counter.kicad_sch (KiCad schematic)
At the start: 12 parts, among them U301 74HC74, U302 74HC74

Commit message: Routing quickly
Parts:
- added R305: 100k, Resistor_THT:R_Axial_DIN0207_L6.3mm_D2.5mm_P7.62mm_Horizontal, symbol Device:R
- added SW201: SW_Push, Button_Switch_THT:SW_PUSH_6mm_H4.3mm, symbol Switch:SW_Push
Connections:
- net +5V: now also R305.1
- net CLK: now also U301.11 (C); no longer U301.3 (C)
- net GND: now also SW201.2
- net Out0: now also U301.9 (Q); no longer U301.5 (Q)
- net Out1: now also U301.5 (Q); no longer U301.9 (Q)
- net Out2: now also U302.9 (Q); no longer U302.5 (Q)
- net Out3: now also U302.5 (Q); no longer U302.9 (Q)
- net ~{Q_{0}}: now also U301.12 (D), U301.3 (C), U301.8 (~{Q}); no longer U301.11 (C), U301.2 (D), U301.6 (~{Q})
- net ~{Q_{1}}: now also U301.2 (D), U301.6 (~{Q}), U302.11 (C); no longer U301.12 (D), U301.8 (~{Q}), U302.3 (C)
- net ~{Q_{2}}: now also U302.12 (D), U302.3 (C), U302.8 (~{Q}); no longer U302.11 (C), U302.2 (D), U302.6 (~{Q})
- net ~{Q_{3}}: now also U302.2 (D), U302.6 (~{Q}); no longer U302.12 (D), U302.8 (~{Q})
- net ~{RESET}: now also R305.2, SW201.1
Other:
- moved on the sheet: U301A, U301B, U302A, U302B
