File: Chained 4017/triple4017.kicad_sch (KiCad schematic)
At the start: 4 parts, among them U301 4017, U302 4017, U303 4017, U304 74HC00

Commit message: Roughing out PCB layout
Parts:
- U304: footprint (none) -> Package_DIP:DIP-14_W7.62mm_Socket
Changed lines of the file:
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@@
       (effects (font (size 1.27 1.27)) (justify left))
     )
-    (property "Footprint" "" (at 33.02 168.91 0)
+    (property "Footprint" "Package_DIP:DIP-14_W7.62mm_Socket" (at 33.02 168.91 0)
       (effects (font (size 1.27 1.27)) hide)
     )
@@
       (effects (font (size 1.27 1.27)))
     )
-    (property "Footprint" "" (at 175.26 88.9 0)
+    (property "Footprint" "Package_DIP:DIP-14_W7.62mm_Socket" (at 175.26 88.9 0)
       (effects (font (size 1.27 1.27)) hide)
     )
@@
       (effects (font (size 1.27 1.27)))
     )
-    (property "Footprint" "" (at 91.44 88.9 0)
+    (property "Footprint" "Package_DIP:DIP-14_W7.62mm_Socket" (at 91.44 88.9 0)
       (effects (font (size 1.27 1.27)) hide)
     )
@@
       (effects (font (size 1.27 1.27)))
     )
-    (property "Footprint" "" (at 157.48 88.9 0)
+    (property "Footprint" "Package_DIP:DIP-14_W7.62mm_Socket" (at 157.48 88.9 0)
       (effects (font (size 1.27 1.27)) hide)
     )
@@
       (effects (font (size 1.27 1.27)))
     )
-    (property "Footprint" "" (at 73.66 88.9 0)
-      (effects (font (size 1.27 1.27)) hide)
-    )
+    (property "Footprint" "Package_DIP:DIP-14_W7.62mm_Socket" (at 73.66 88.9 0)
+      (effects (font (size 1.27 1.27)) hide)
+    )

Commit message: More layout
Parts:
- added D301, D302, D303, D304: LED, LED_THT:LED_D3.0mm, symbol Device:LED
- added R301, R302, R303, R304: R, Resistor_THT:R_Axial_DIN0207_L6.3mm_D2.5mm_P7.62mm_Horizontal, symbol Device:R
Connections:
- net GND: now also R301.2, R302.2, R303.2, R304.2
- net Q9_{1}: now reaches U302.11 (Q9), U302.13 (CKEN), U304.9
- net Q9_{1}: now also D302.2 (A)
- net Q9_{2}: now reaches U301.15 (Reset), U303.11 (Q9)
- net Q9_{2}: now also D303.2 (A)
- net Q0_{1}: now reaches U302.3 (Q0), U303.15 (Reset)
- net Q0_{1}: now also D304.2 (A)
- net Q9_{0}: now reaches U301.11 (Q9), U301.13 (CKEN), U304.1
- net Q9_{0}: now also D301.2 (A)
- new net: D303.1 (K), R303.1
- new net: D304.1 (K), R304.1
- new net: D302.1 (K), R302.1
- new net: D301.1 (K), R301.1

Commit message: Layout and starting routing
Connections:
- net Out5: no longer U301.10 (Q4)
- new net Out4: U301.10 (Q4)
Changed lines of the file:
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@@
     (stroke (width 0) (type default))
   )
-  (label "Out5" (at 48.26 68.58 90) (fields_autoplaced)
+  (label "Out4" (at 48.26 68.58 90) (fields_autoplaced)
     (effects (font (size 1.27 1.27)) (justify left bottom))
   )

Commit message: Capacitors and routing
Parts:
- added C802 (x4): 0.1u, Capacitor_THT:C_Disc_D4.3mm_W1.9mm_P5.00mm, symbol Device:C
Connections:
- net +5V: now also C802.2, C802.2, C802.2, C802.2
- net CLK: now also U304.5; no longer U304.10
- net GND: now also C802.1, C802.1, C802.1, C802.1
- net Q9_{1}: now also U304.4; no longer U304.9
- net at U304.11: now also U302.14 (CLK); no longer U303.14 (CLK)
- net at U304.12, U304.13: now also U304.3; no longer U304.8
- net at U304.6: now also U304.10, U304.9; no longer U302.14 (CLK)
- new net: U303.14 (CLK), U304.8
Other:
- moved on the sheet: U304B, U304C, U304D
