File: CrankGPT Power/CrankGPT Power.kicad_pcb (KiCad board)
At the start: 2 copper layers, 9 parts, among them J101 USB_A, U1 MIC29502WT

Commit message: Roughing out
Parts:
- removed J101: USB_A, Connector_USB:USB_A_Molex_67643_Horizontal
- added C1: MAL222091008E3, Capacitor_THT:CP_Radial_D18.0mm_P7.50mm, F.Cu at (50.0, 50.0)
- added C2: MAL222091008E3, Capacitor_THT:CP_Radial_D18.0mm_P7.50mm, F.Cu at (50.0, 72.5)
- added C3: MAL222091008E3, Capacitor_THT:CP_Radial_D18.0mm_P7.50mm, F.Cu at (50.0, 95.0)
- added C7: 2200u, Capacitor_THT:CP_Radial_D10.0mm_P5.00mm, F.Cu at (110.0, 100.0)
- added H1: MountingHole, MountingHole:MountingHole_2.7mm_M2.5, F.Cu at (27.5, 107.5)
- added H2: MountingHole, MountingHole:MountingHole_2.7mm_M2.5, F.Cu at (132.5, 110.0)
- added H3: MountingHole, MountingHole:MountingHole_2.7mm_M2.5, F.Cu at (78.0, 134.4)
- added H4: MountingHole, MountingHole:MountingHole_2.7mm_M2.5, F.Cu at (78.0, 141.3)
- added J1: Conn_01x02_Pin, Connector_PinHeader_2.54mm:PinHeader_1x02_P2.54mm_Vertical, F.Cu at (27.5, 77.5)
- added J2: Conn_01x02_Pin, Connector_PinHeader_2.54mm:PinHeader_1x02_P2.54mm_Vertical, F.Cu at (130.0, 100.0)
- added J4: Conn_01x02_Socket, Connector_JST:JST_NV_B02P-NV_1x02_P5.00mm_Vertical, F.Cu at (31.3, 54.3)
- added J5: USB_A, Connector_USB:USB_A_Molex_67643_Horizontal, F.Cu at (122.5, 55.0)
- added R4: 2k2, Resistor_THT:R_Axial_DIN0207_L6.3mm_D2.5mm_P7.62mm_Horizontal, F.Cu at (115.0, 58.7)
- added R5: 1k, Resistor_THT:R_Axial_DIN0207_L6.3mm_D2.5mm_P7.62mm_Horizontal, F.Cu at (115.0, 72.5)
- added R6: 1k, Resistor_THT:R_Axial_DIN0207_L6.3mm_D2.5mm_P7.62mm_Horizontal, F.Cu at (115.0, 82.5)
- added SW1: SW_SPDT, Button_Switch_THT:SW_Slide_SPDT_Angled_CK_OS102011MA1Q, F.Cu at (105.4, 37.5)
- moved U1 39.1 mm to (102.5, 55.0), turned to 90 degrees
- moved R3 22.7 mm to (90.0, 90.0)
- moved R2 22.6 mm to (90.0, 67.5)
- moved R1 22.5 mm to (90.0, 45.0)
- moved C6 21.9 mm to (72.5, 95.0)
- moved C5 21.8 mm to (72.5, 72.5)
- moved C4 21.7 mm to (72.5, 50.0)
- moved D1 21.6 mm to (37.6, 40.0), turned to 180 degrees
- renumbered C1 to C4, C2 to C5, C3 to C6
Connections:
- D1 pad 2: unconnected-(D1-A-Pad2) -> /V_{in}
- U1 pad 4: unconnected-(U1-VOUT-Pad4) -> /V_{out}
- U1 pad 5: unconnected-(U1-ADJ-Pad5) -> Net-(U1-ADJ)
Other:
- board outline added: 112.5 x 77.5 mm

Commit message: Experimenting a little
Other:
- board text added: "JLCJLCJLCJLC"
- board text added: "RGE2026"
Changed lines of the file:
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@@
 		(layer "Edge.Cuts")
+	)
+	(gr_text "RGE2026"
+		(at 37.5 65 90)
+		(layer "B.Cu")
+		(effects
+			(font
+				(size 3 3)
+				(thickness 0.5)
+				(bold yes)
+			)
+			(justify left bottom mirror)
+		)
+	)
+	(gr_text "JLCJLCJLCJLC"
+		(at 127.5 95 0)
+		(layer "B.SilkS")
+		(effects
+			(font
+				(size 3 3)
+				(thickness 0.5)
+				(bold yes)
+			)
+			(justify left bottom mirror)
+		)
 	)
 	(embedded_fonts no)

Commit message: Laying out
Parts:
- added C8: 2200u, Capacitor_THT:CP_Radial_D10.0mm_P5.00mm, F.Cu at (102.0, 95.0)
- added J3: Conn_01x02_Pin, Connector_PinHeader_2.54mm:PinHeader_1x02_P2.54mm_Vertical, F.Cu at (117.0, 95.0)
- C7: value 2200u -> 0.1u; footprint Capacitor_THT:CP_Radial_D10.0mm_P5.00mm -> Capacitor_THT:C_Disc_D4.3mm_W1.9mm_P5.00mm
- J2: value Conn_01x02_Pin -> Conn_01x02_Socket; footprint Connector_PinHeader_2.54mm:PinHeader_1x02_P2.54mm_Vertical -> Connector_JST:JST_NV_B02P-NV_1x02_P5.00mm_Vertical
- moved J2 111.9 mm to (27.5, 55.0), turned to 90 degrees
- moved H4 108.6 mm to (117.0, 40.0)
- moved H3 107.3 mm to (27.0, 40.0)
- moved J4 85.8 mm to (117.0, 50.0)
- moved C7 38.6 mm to (96.0, 64.0), turned to 90 degrees
- moved J5 28.7 mm to (108.5, 80.0)
- moved J1 17.5 mm to (27.5, 95.0)
- moved R4 16.6 mm to (102.0, 69.0), turned to 180 degrees
- moved H2 15.8 mm to (117.0, 107.0)
- moved R6 13.5 mm to (102.0, 79.0), turned to 180 degrees
- moved R5 13.1 mm to (102.0, 74.0), turned to 180 degrees
- moved D1 10.0 mm to (37.5, 50.0), turned to -90 degrees
- moved SW1 7.92 mm to (97.5, 38.0)
- moved U1 2.50 mm to (100.0, 55.0)
- moved H1 0.71 mm to (27.0, 107.0)
Connections:
- C7 pad 1: /V_{out} -> GND
- C7 pad 2: GND -> Net-(D1-K)
- J2 pad 1: /V_{out} -> GND
- J2 pad 2: GND -> /V_{in}
- J4 pad 1: /V_{in} -> /V_{out}
- R5 pad 1: Net-(R4-Pad2) -> Net-(U1-ADJ)
- R5 pad 2: Net-(U1-ADJ) -> Net-(R4-Pad2)
- SW1 pad 1: Net-(SW1-A) -> GND
- SW1 pad 2: Net-(D1-K) -> Net-(SW1-B)
- SW1 pad 3: unconnected-(SW1-C-Pad3) -> Net-(D1-K)
- U1 pad 1: Net-(SW1-A) -> Net-(SW1-B)
Routing:
- net Net-(C1-Pad2): track 0.00 -> 116.7 mm
- net Net-(C2-Pad2): track 0.00 -> 116.7 mm
- net Net-(U1-ADJ): track 0.00 -> 50.3 mm
- net Net-(SW1-B): track 0.00 -> 21.2 mm
- net Net-(D1-K): track 0.00 -> 10.2 mm
- net Net-(R4-Pad2): track 0.00 -> 5.00 mm
- net Net-(J5-D+): track 0.00 -> 2.00 mm
- net GND: vias 0 -> 3
- added copper zone on B.Cu, net /V_{in}
- added copper zone on B.Cu, net /V_{out}
- added copper zone on B.Cu, net GND
- added copper zone on F.Cu, net GND
- added copper zone on B.Cu, net Net-(D1-K)
Other:
- board size 112.5 x 77.5 mm -> 100 x 77 mm
- board text added: "GND"

Commit message: Shrink board slightly
Parts:
- moved H1 2.00 mm to (27.0, 105.0)
- moved H2 2.00 mm to (117.0, 105.0)
Other:
- board size 100 x 77 mm -> 100 x 75 mm

Commit message: Correct diode footprint
Parts:
- D1: footprint Diode_THT:D_DO-41_SOD81_P10.16mm_Horizontal -> Diode_THT:D_P600_R-6_P20.00mm_Horizontal
- moved C1 5.00 mm to (55.0, 50.0)
- moved C2 5.00 mm to (55.0, 72.5)
- moved C3 5.00 mm to (55.0, 95.0)
- moved C4 3.50 mm to (76.0, 50.0)
- moved C5 3.50 mm to (76.0, 72.5)
- moved C6 3.50 mm to (76.0, 95.0)
- moved D1 2.50 mm to (40.0, 50.0)
Routing:
- net Net-(D1-K): track 10.2 -> 64.6 mm
- net Net-(C2-Pad2): track 116.7 -> 85.6 mm
- net Net-(C1-Pad2): track 116.7 -> 98.8 mm
