File: CrankGPT Power/CrankGPT Power.kicad_sch (KiCad schematic)
At the start: 1 part

Commit message: Adding some components
Parts:
- added C1, C2, C3: MAL222091008E3, Capacitor_THT:CP_Radial_D18.0mm_P7.50mm, symbol Device:C_Polarized
- added J101: USB_A, Connector_USB:USB_A_Molex_67643_Horizontal, symbol Connector:USB_A
- added R1, R2, R3: RSF100JR-73-100R, Resistor_THT:R_Axial_DIN0414_L11.9mm_D4.5mm_P15.24mm_Horizontal, symbol Device:R
- added SW1: SW_SPDT, symbol Switch:SW_SPDT
- added U1: MIC29502WT, Package_TO_SOT_THT:TO-220-5_P3.4x3.7mm_StaggerEven_Lead3.8mm_Vertical, symbol Regulator_Linear:MIC29502WT
- D1: value D_Schottky -> 15SQ045
Connections:
- net at D1.1 (K): now also C1.1, R1.1, SW1.2 (B), U1.2 (VIN)
- new net: SW1.1 (A), U1.1 (EN)
- new net: C2.2, C3.1, R2.2, R3.1
- new net: C1.2, C2.1, R1.2, R2.1
- new net GND: C3.2, R3.2, U1.3 (GND)
- no-connect marks 0 -> 1
Other:
- moved on the sheet: D1

Commit message: Roughing out
Parts:
- removed J101: USB_A, Connector_USB:USB_A_Molex_67643_Horizontal, symbol Connector:USB_A
- added C1, C2, C3: MAL222091008E3, Capacitor_THT:CP_Radial_D18.0mm_P7.50mm, symbol Device:C_Polarized
- added C7: 2200u, Capacitor_THT:CP_Radial_D10.0mm_P5.00mm, symbol Device:C_Polarized
- added H1, H2, H3, H4: MountingHole, MountingHole:MountingHole_2.7mm_M2.5, symbol Mechanical:MountingHole
- added J1, J2: Conn_01x02_Pin, Connector_PinHeader_2.54mm:PinHeader_1x02_P2.54mm_Vertical, symbol Connector:Conn_01x02_Pin
- added J4: Conn_01x02_Socket, Connector_JST:JST_NV_B02P-NV_1x02_P5.00mm_Vertical, symbol Connector:Conn_01x02_Socket
- added J5: USB_A, Connector_USB:USB_A_Molex_67643_Horizontal, symbol Connector:USB_A
- added R4: 2k2, Resistor_THT:R_Axial_DIN0207_L6.3mm_D2.5mm_P7.62mm_Horizontal, symbol Device:R
- added R5, R6: 1k, Resistor_THT:R_Axial_DIN0207_L6.3mm_D2.5mm_P7.62mm_Horizontal, symbol Device:R
- SW1: footprint (none) -> Button_Switch_THT:SW_Slide_SPDT_Angled_CK_OS102011MA1Q
- renumbered C1 to C4, C2 to C5, C3 to C6
Connections:
- net GND: now also C3.2, C7.2, J1.2 (Pin_2), J2.2 (Pin_2), J4.2 (Pin_2), J5.4 (GND), R6.2
- net at C4.1, D1.1 (K), R1.1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: now also C1.1
- net V_{out}: now reaches U1.4 (VOUT)
- net V_{out}: now also C7.1, J2.1 (Pin_1), J5.1 (VBUS), R4.1
- net at U1.5 (ADJ): now also R5.2, R6.1
- net V_{in}: now reaches D1.2 (A)
- net V_{in}: now also J1.1 (Pin_1), J4.1 (Pin_1)
- net at C5.2, C6.1, R2.2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: now also C2.2, C3.1
- net at C4.2, C5.1, R1.2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: now also C1.2, C2.1
- new net: R4.2, R5.1
- new net: J5.2 (D-), J5.3 (D+)
- no-connect marks 1 -> 2
Other:
- moved on the sheet: C4, C5, C6, D1, R1, R2, R3, SW1, U1

Commit message: Laying out
Parts:
- added C7: 0.1u, Capacitor_THT:C_Disc_D4.3mm_W1.9mm_P5.00mm, symbol Device:C
- added J4: Conn_01x02_Socket, Connector_JST:JST_NV_B02P-NV_1x02_P5.00mm_Vertical, symbol Connector:Conn_01x02_Socket
- renumbered C7 to C8, J4 to J2, J2 to J3
Connections:
- net GND: now also J2.1 (Pin_1), SW1.1 (A), C7.1, J4.2 (Pin_2); no longer J2.2 (Pin_2)
- net V_{in}: now also J2.2 (Pin_2); no longer J2.1 (Pin_1)
- net V_{out}: now also J4.1 (Pin_1)
- net at U1.1 (EN): now also SW1.2 (B); no longer SW1.1 (A)
- net at C1.1, C4.1, D1.1 (K)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: now also SW1.3 (C), C7.2; no longer SW1.2 (B)
- net at R6.1, U1.5 (ADJ): now also R5.1; no longer R5.2
- net at R4.2: now also R5.2; no longer R5.1
- no-connect marks 2 -> 1
Other:
- moved on the sheet: J3, R5, SW1

Commit message: Correct diode footprint
Parts:
- D1: footprint Diode_THT:D_DO-41_SOD81_P10.16mm_Horizontal -> Diode_THT:D_P600_R-6_P20.00mm_Horizontal
Changed lines of the file:
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@@
 			)
 		)
-		(property "Footprint" "Diode_THT:D_DO-41_SOD81_P10.16mm_Horizontal"
+		(property "Footprint" "Diode_THT:D_P600_R-6_P20.00mm_Horizontal"
 			(at 41.91 50.8 0)
 			(hide yes)
